File: hardware/foras-promineo-FM/SLI-Backplane-Blank-Card-KiCad.kicad_sch (KiCad schematic)
At the start: 29 parts, among them J201 TSM-102-01-L-SV-P-TR, P1 Card Edge for HSEC8-160-01-S-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, Q204 MMBT3906-7-F, Q205 MMBT4401-7-F, Q206 IRF7458, Q207 IRF7404, Q208 IRF7458, Q210 MMBT4401-7-F, Q211 IRF7404, Q212 IRF7404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

Commit message: lots of stuff
Parts:
- removed D204, D205, D? (x3): 1N4148WSTR, Diode_SMD:D_SOD-323, symbol mainboard-rescue:D-Device-mainboard-rescue
- removed Q204: MMBT3906-7-F, Package_TO_SOT_SMD:SOT-23, symbol mainboard-rescue:Q_PNP_BEC-Device-mainboard-rescue
- removed Q210: MMBT4401-7-F, Package_TO_SOT_SMD:SOT-23, symbol mainboard-rescue:Q_NPN_BCE-Device-mainboard-rescue
- removed R212, R215: 100k, Resistor_SMD:R_0603_1608Metric, symbol mainboard-rescue:R_US-Device-mainboard-rescue
- removed R247, R?: 2.2Meg, Resistor_SMD:R_0603_1608Metric, symbol mainboard-rescue:R_US-Device-mainboard-rescue
- added Q? (x3): MMBT3906-7-F, Package_TO_SOT_SMD:SOT-23, symbol mainboard-rescue:Q_PNP_BEC-Device-mainboard-rescue
- added R?: 2.2Meg, Resistor_SMD:R_0603_1608Metric, symbol mainboard-rescue:R_US-Device-mainboard-rescue
- added R?: 100k, symbol Device:R_US
- added R?: 100k, Resistor_SMD:R_0603_1608Metric, symbol mainboard-rescue:R_US-Device-mainboard-rescue
- added R?: 2.2Meg, symbol Device:R_US
- R213, R218: value 4.7k -> 100k
- R214, R216, R219, R220, R221, R248: value 100k -> 2.2Meg
Connections:
- net 5V_USB: now also R214.1, R?.1; no longer R218.2
- net RBF: now also R218.2, R?.2; no longer Q206.4 (G), Q220.4 (G), R214.2, R248.2
- net SEP1: now also R?.2
- net VBUS_INHIBIT: now also R220.1, R221.1, Q?.2 (E), Q?.2 (E)
- net VBUS_USB: now also R219.1
- net VCHRG_USB: now also R216.1
- net at Q208.4 (G): now also Q?.3 (C), R?.1
- net at Q213.4 (G), R219.2: now also Q?.2 (E)
- net at R218.1: now also Q?.1 (B)
- removed net Debug_Inhibit_Vcc: R214.1, R216.1, R219.1
- removed net Inhibit_Vcc: R220.1, R221.1, R248.1
- net VBATT_RET renamed GNDREF
- net GNDREF: now also R214.2, R248.2, Q?.3 (C), R?.2
- new net: Q206.4 (G), R?.2
- new net: Q220.4 (G), Q?.3 (C), R248.1
- new net: Q?.1 (B), R?.1 (x2)
Other:
- note added: "(RBF open) & (sep1 open) & (sep2 open) & (sep3 open) = main bus powered"
- note added: "GNDREF is battery return"
- note added: "RBF is N/O to gnd (install pulls RBF low)"
- note added: "Vbatt_RET"
- note added: "installing this jumper will allow data but disable usb source"
- note added: "sep switches are N/C to GND (switch press opens circuit; i.e. in deployer)"
- note removed: "AOZ1327DI-01"
- note removed: "DNP"
- note removed: "RBF is N/O to gnd when removed"
- note removed: "RBF is NO to gnd when removed"
- note removed: "Sep switches are N/O to GND"
- note removed: "Sep_Sw_Vcc is an OR of solar and batt inputs, allowing either to enable the bus"
- note removed: "ZXMS6005DGTA"
- note removed: "current flow"
- note removed: "double check this circuit tmmr"
- note removed: "flipped, update in PCB"
- note removed: "if gndref is d/c from gnd these resistors allow a refrence to still be made to turn the fets on"
- note removed: "installing jumper will allow data but disable usb pwr sourcing"
- note removed: "look into just replacing debug inhibits with jumpers"
- note removed: "the need to pull the pmos' high during the whole operation of the sat will just waste power and add extra falue modes"
- note removed: "vbatt voltage & RBF removed & (sep1 low) & (sep2 low) & (sep3 low) = main bus powered"
- moved on the sheet: J201, Q205, Q206, Q207, Q208, Q211, Q212, Q213, Q220, R213, R214, R216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
