File: hardware/foras-promineo-revB-fm/5V_regulator.kicad_sch (KiCad schematic)
At the start: 15 parts, among them Q222 MMBT3906-7-F, U210 TPS63070

Commit message: fm sch changes
Parts:
- added R114: 10k, Resistor_SMD:R_0603_1608Metric, symbol Device:R_US
- added TH51: 10k, Resistor_SMD:R_0603_1608Metric, symbol Device:Thermistor_NTC_US
- C235, C236, C237, C238, C239, C240, C241: symbol mainboard-rescue:C-Device-mainboard-rescue -> Device:C
- L202: symbol mainboard-rescue:L-Device-mainboard-rescue -> Device:L
- R251, R252, R253, R254, R255: symbol mainboard-rescue:R_US-Device-mainboard-rescue -> Device:R_US
Connections:
- net GND: now also TH51.2
- new net 3.3V: R114.1
- new net NTC: R114.2, TH51.1
Changed lines of the file:
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@@
   (junction (at 97.79 83.82) (diameter 0) (color 0 0 0 0)
   )
+  (junction (at 142.24 105.41) (diameter 0) (color 0 0 0 0)
+  )
   (junction (at 213.36 60.96) (diameter 0) (color 0 0 0 0)
   )
@@
     (stroke (width 0) (type default) (color 0 0 0 0))
   )
+  (wire (pts (xy 142.24 95.25) (xy 142.24 97.79))
+    (stroke (width 0) (type default) (color 0 0 0 0))
+  )
   (wire (pts (xy 180.34 69.85) (xy 180.34 76.2))
     (stroke (width 0) (type default) (color 0 0 0 0))
@@
     (stroke (width 0) (type default) (color 0 0 0 0))
   )
+  (wire (pts (xy 142.24 105.41) (xy 142.24 106.68))
+    (stroke (width 0) (type default) (color 0 0 0 0))
+  )
   (wire (pts (xy 119.38 59.69) (xy 146.05 59.69))
     (stroke (width 0) (type default) (color 0 0 0 0))
@@
   )
   (wire (pts (xy 180.34 60.96) (xy 191.77 60.96))
+    (stroke (width 0) (type default) (color 0 0 0 0))
+  )
+  (wire (pts (xy 142.24 105.41) (xy 157.48 105.41))
     (stroke (width 0) (type default) (color 0 0 0 0))
   )
@@
     )
   )
+  (global_label "3.3V" (shape bidirectional) (at 142.24 95.25 0) (fields_autoplaced)
+    (effects (font (size 1.27 1.27)) (justify left))
+    (property "Intersheet References" "${INTERSHEET_REFS}" (id 0) (at 1.27 -30.48 0)
+      (effects (font (size 1.27 1.27)) hide)
+    )
+  )
   (global_label "VBUS" (shape bidirectional) (at 91.44 68.58 180) (fields_autoplaced)
     (effects (font (size 1.27 1.27)) (justify right))
@@
   )
   (hierarchical_label "Vout" (shape input) (at 227.33 60.96 0)
+    (effects (font (size 1.27 1.27)) (justify left))
+  )
+  (hierarchical_label "NTC" (shape input) (at 157.48 105.41 0)
     (effects (font (size 1.27 1.27)) (justify left))
   )
@@
     (pin "9")
   )
-  (symbol (lib_id "mainboard-rescue:R_US-Device-mainboard-rescue") (at 97.79 88.9 0) (unit 1)
+  (symbol (lib_id "Device:R_US") (at 97.79 88.9 0) (unit 1)
     (in_bom yes) (on_board yes)
     (property "Reference" "R255" (id 0) (at 99.5172 87.7316 0)
@@
     (pin "1")
   )
-  (symbol (lib_id "mainboard-rescue:C-Device-mainboard-rescue") (at 127 67.31 180) (unit 1)
+  (symbol (lib_id "Device:C") (at 127 67.31 180) (unit 1)
     (in_bom yes) (on_board yes)
     (property "Reference" "C241" (id 0) (at 129.921 66.1416 0)
@@
     (pin "2")
   )
-  (symbol (lib_id "mainboard-rescue:C-Device-mainboard-rescue") (at 115.57 53.34 0) (unit 1)
+  (symbol (lib_id "Device:C") (at 115.57 53.34 0) (unit 1)
     (in_bom yes) (on_board yes)
     (property "Reference" "C237" (id 0) (at 118.491 52.1716 0)
@@
     (pin "2")
   )
-  (symbol (lib_id "mainboard-rescue:C-Device-mainboard-rescue") (at 104.14 53.34 0) (unit 1)
+  (symbol (lib_id "Device:C") (at 104.14 53.34 0) (unit 1)
     (in_bom yes) (on_board yes)
     (property "Reference" "C236" (id 0) (at 107.061 52.1716 0)
@@
     (pin "2")
   )
-  (symbol (lib_id "mainboard-rescue:C-Device-mainboard-rescue") (at 92.71 53.34 0) (unit 1)
+  (symbol (lib_id "Device:C") (at 92.71 53.34 0) (unit 1)
     (in_bom yes) (on_board yes)
     (property "Reference" "C235" (id 0) (at 95.631 52.1716 0)
@@
     (pin "1")
   )
-  (symbol (lib_id "mainboard-rescue:L-Device-mainboard-rescue") (at 170.18 52.07 0) (unit 1)
+  (symbol (lib_id "Device:L") (at 170.18 52.07 0) (unit 1)
     (in_bom yes) (on_board yes)
     (property "Reference" "L202" (id 0) (at 171.5262 50.9016 0)
@@
     (pin "2")
   )
-  (symbol (lib_id "mainboard-rescue:R_US-Device-mainboard-rescue") (at 180.34 64.77 0) (unit 1)
+  (symbol (lib_id "Device:R_US") (at 180.34 64.77 0) (unit 1)
     (in_bom yes) (on_board yes)
     (property "Reference" "R251" (id 0) (at 182.0672 63.6016 0)
@@
     (pin "2")
   )
-  (symbol (lib_id "mainboard-rescue:R_US-Device-mainboard-rescue") (at 180.34 80.01 0) (unit 1)
+  (symbol (lib_id "Device:R_US") (at 180.34 80.01 0) (unit 1)
     (in_bom yes) (on_board yes)
     (property "Reference" "R254" (id 0) (at 182.0672 78.8416 0)
@@
     (pin "1")
   )
-  (symbol (lib_id "mainboard-rescue:R_US-Device-mainboard-rescue") (at 191.77 68.58 0) (unit 1)
+  (symbol (lib_id "Device:R_US") (at 191.77 68.58 0) (unit 1)
     (in_bom yes) (on_board yes)
     (property "Reference" "R252" (id 0) (at 193.4972 67.4116 0)
@@
     (pin "2")
   )
-  (symbol (lib_id "mainboard-rescue:C-Device-mainboard-rescue") (at 201.93 64.77 0) (unit 1)
+  (symbol (lib_id "Device:C") (at 201.93 64.77 0) (unit 1)
     (in_bom yes) (on_board yes)
     (property "Reference" "C238" (id 0) (at 204.851 63.6016 0)
@@
     (pin "2")
   )
-  (symbol (lib_id "mainboard-rescue:C-Device-mainboard-rescue") (at 213.36 64.77 0) (unit 1)
+  (symbol (lib_id "Device:C") (at 213.36 64.77 0) (unit 1)
     (in_bom yes) (on_board yes)
     (property "Reference" "C239" (id 0) (at 216.281 63.6016 0)
@@
     (pin "1")
   )
-  (symbol (lib_id "mainboard-rescue:C-Device-mainboard-rescue") (at 223.52 64.77 0) (unit 1)
+  (symbol (lib_id "Device:C") (at 223.52 64.77 0) (unit 1)
     (in_bom yes) (on_board yes)
     (property "Reference" "C240" (id 0) (at 226.441 63.6016 0)
@@
     (pin "1")
   )
-  (symbol (lib_id "mainboard-rescue:R_US-Device-mainboard-rescue") (at 85.09 77.47 270) (unit 1)
+  (symbol (lib_id "Device:R_US") (at 85.09 77.47 270) (unit 1)
     (in_bom yes) (on_board yes)
     (property "Reference" "R253" (id 0) (at 85.09 72.263 90))
@@
     (pin "2")
   )
+  (symbol (lib_id "Device:Thermistor_NTC_US") (at 142.24 110.49 0) (unit 1)
+    (in_bom yes) (on_board yes) (fields_autoplaced)
+    (property "Reference" "TH51" (id 0) (at 144.78 109.5374 0)
+      (effects (font (size 1.27 1.27)) (justify left))
+    )
+    (property "Value" "10k" (id 1) (at 144.78 112.0774 0)
+      (effects (font (size 1.27 1.27)) (justify left))
+    )
+    (property "Footprint" "Resistor_SMD:R_0603_1608Metric" (id 2) (at 142.24 109.22 0)
+      (effects (font (size 1.27 1.27)) hide)
+    )
+    (property "Datasheet" "~" (id 3) (at 142.24 109.22 0)
+      (effects (font (size 1.27 1.27)) hide)
+    )
+    (pin "1")
+    (pin "2")
+  )
+  (symbol (lib_id "Device:R_US") (at 142.24 101.6 0) (unit 1)
+    (in_bom yes) (on_board yes) (fields_autoplaced)
+    (property "Reference" "R114" (id 0) (at 144.78 100.3299 0)
+      (effects (font (size 1.27 1.27)) (justify left))
+    )
+    (property "Value" "10k" (id 1) (at 144.78 102.8699 0)
+      (effects (font (size 1.27 1.27)) (justify left))
+    )
+    (property "Footprint" "Resistor_SMD:R_0603_1608Metric" (id 2) (at 143.256 101.854 90)
+      (effects (font (size 1.27 1.27)) hide)
+    )
+    (property "Datasheet" "~" (id 3) (at 142.24 101.6 0)
+      (effects (font (size 1.27 1.27)) hide)
+    )
+    (pin "1")
+    (pin "2")
+  )
+  (symbol (lib_id "mainboard:GND") (at 142.24 116.84 0) (unit 1)
+    (in_bom yes) (on_board yes)
+    (property "Reference" "#GND0117" (id 0) (at 142.24 116.84 0)
+      (effects (font (size 1.27 1.27)) hide)
+    )
+    (property "Value" "GND" (id 1) (at 142.24 119.9134 0)
+      (effects (font (size 1.4986 1.4986)))
+    )
+    (property "Footprint" "" (id 2) (at 142.24 116.84 0)
+      (effects (font (size 1.27 1.27)) hide)
+    )
+    (property "Datasheet" "" (id 3) (at 142.24 116.84 0)
+      (effects (font (size 1.27 1.27)) hide)
+    )
+    (pin "1")
+  )
 )
