File: hardware/foras-promineo-revB-fm/Blank-Card-Default.kicad_sch (KiCad schematic)
At the start: 39 parts, among them J200 ZX62-AB-5PA(31), Q200 BC847BM3T5G, Q201 BC847BM3T5G, Q202 BC847BM3T5G, Q203 BC847BM3T5G, SW200 SW_Push_SPST, U200 AP2161W

Commit message: fm sch changes
Parts:
- C200, C201, C202, C203, C204, C205, C206, C207, C208, C209: symbol mainboard-rescue:C-Device-mainboard-rescue -> Device:C
- R200, R201, R202, R203, R204, R205, R206, R207, R208, R209, R210, R211: symbol mainboard-rescue:R_US-Device-mainboard-rescue -> Device:R_US
Changed lines of the file:
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@@
     (effects (font (size 1.27 1.27)) (justify right))
   )
-  (symbol (lib_id "mainboard-rescue:R_US-Device-mainboard-rescue") (at 176.53 64.77 0) (unit 1)
+  (symbol (lib_id "Device:R_US") (at 176.53 64.77 0) (unit 1)
     (in_bom yes) (on_board yes)
     (property "Reference" "R211" (id 0) (at 178.2572 63.6016 0)
@@
     (pin "6")
   )
-  (symbol (lib_id "mainboard-rescue:R_US-Device-mainboard-rescue") (at 90.17 68.58 0) (unit 1)
+  (symbol (lib_id "Device:R_US") (at 90.17 68.58 0) (unit 1)
     (in_bom yes) (on_board yes)
     (property "Reference" "R201" (id 0) (at 91.8972 67.4116 0)
@@
     (pin "2")
   )
-  (symbol (lib_id "mainboard-rescue:C-Device-mainboard-rescue") (at 80.01 68.58 0) (unit 1)
+  (symbol (lib_id "Device:C") (at 80.01 68.58 0) (unit 1)
     (in_bom yes) (on_board yes)
     (property "Reference" "C205" (id 0) (at 82.931 67.4116 0)
@@
     (pin "2")
   )
-  (symbol (lib_id "mainboard-rescue:C-Device-mainboard-rescue") (at 68.58 68.58 0) (unit 1)
+  (symbol (lib_id "Device:C") (at 68.58 68.58 0) (unit 1)
     (in_bom yes) (on_board yes)
     (property "Reference" "C204" (id 0) (at 71.501 67.4116 0)
@@
     (pin "5")
   )
-  (symbol (lib_id "mainboard-rescue:R_US-Device-mainboard-rescue") (at 207.01 50.8 0) (unit 1)
+  (symbol (lib_id "Device:R_US") (at 207.01 50.8 0) (unit 1)
     (in_bom yes) (on_board yes)
     (property "Reference" "R200" (id 0) (at 208.7372 49.6316 0)
@@
     (pin "2")
   )
-  (symbol (lib_id "mainboard-rescue:C-Device-mainboard-rescue") (at 240.03 60.96 0) (unit 1)
+  (symbol (lib_id "Device:C") (at 240.03 60.96 0) (unit 1)
     (in_bom yes) (on_board yes)
     (property "Reference" "C202" (id 0) (at 242.951 59.7916 0)
@@
     (pin "2")
   )
-  (symbol (lib_id "mainboard-rescue:R_US-Device-mainboard-rescue") (at 102.87 99.06 0) (unit 1)
+  (symbol (lib_id "Device:R_US") (at 102.87 99.06 0) (unit 1)
     (in_bom yes) (on_board yes)
     (property "Reference" "R202" (id 0) (at 104.5972 97.8916 0)
@@
     (pin "3")
   )
-  (symbol (lib_id "mainboard-rescue:R_US-Device-mainboard-rescue") (at 88.9 120.65 270) (unit 1)
+  (symbol (lib_id "Device:R_US") (at 88.9 120.65 270) (unit 1)
     (in_bom yes) (on_board yes)
     (property "Reference" "R206" (id 0) (at 88.9 115.443 90))
@@
     (pin "2")
   )
-  (symbol (lib_id "mainboard-rescue:R_US-Device-mainboard-rescue") (at 151.13 99.06 0) (unit 1)
+  (symbol (lib_id "Device:R_US") (at 151.13 99.06 0) (unit 1)
     (in_bom yes) (on_board yes)
     (property "Reference" "R203" (id 0) (at 152.8572 97.8916 0)
@@
     (pin "2")
   )
-  (symbol (lib_id "mainboard-rescue:R_US-Device-mainboard-rescue") (at 137.16 120.65 270) (unit 1)
+  (symbol (lib_id "Device:R_US") (at 137.16 120.65 270) (unit 1)
     (in_bom yes) (on_board yes)
     (property "Reference" "R207" (id 0) (at 137.16 115.443 90))
@@
     (pin "2")
   )
-  (symbol (lib_id "mainboard-rescue:R_US-Device-mainboard-rescue") (at 199.39 99.06 0) (unit 1)
+  (symbol (lib_id "Device:R_US") (at 199.39 99.06 0) (unit 1)
     (in_bom yes) (on_board yes)
     (property "Reference" "R204" (id 0) (at 201.1172 97.8916 0)
@@
     (pin "2")
   )
-  (symbol (lib_id "mainboard-rescue:R_US-Device-mainboard-rescue") (at 185.42 120.65 270) (unit 1)
+  (symbol (lib_id "Device:R_US") (at 185.42 120.65 270) (unit 1)
     (in_bom yes) (on_board yes)
     (property "Reference" "R208" (id 0) (at 185.42 115.443 90))
@@
     (pin "2")
   )
-  (symbol (lib_id "mainboard-rescue:R_US-Device-mainboard-rescue") (at 248.92 99.06 0) (unit 1)
+  (symbol (lib_id "Device:R_US") (at 248.92 99.06 0) (unit 1)
     (in_bom yes) (on_board yes)
     (property "Reference" "R205" (id 0) (at 250.6472 97.8916 0)
@@
     (pin "2")
   )
-  (symbol (lib_id "mainboard-rescue:R_US-Device-mainboard-rescue") (at 234.95 120.65 270) (unit 1)
+  (symbol (lib_id "Device:R_US") (at 234.95 120.65 270) (unit 1)
     (in_bom yes) (on_board yes)
     (property "Reference" "R209" (id 0) (at 234.95 115.443 90))
@@
     (pin "1")
   )
-  (symbol (lib_id "mainboard-rescue:C-Device-mainboard-rescue") (at 252.73 60.96 0) (unit 1)
+  (symbol (lib_id "Device:C") (at 252.73 60.96 0) (unit 1)
     (in_bom yes) (on_board yes)
     (property "Reference" "C203" (id 0) (at 255.651 59.7916 0)
@@
     (pin "2")
   )
-  (symbol (lib_id "mainboard-rescue:R_US-Device-mainboard-rescue") (at 100.33 168.91 0) (unit 1)
+  (symbol (lib_id "Device:R_US") (at 100.33 168.91 0) (unit 1)
     (in_bom yes) (on_board yes)
     (property "Reference" "R210" (id 0) (at 102.0572 167.7416 0)
@@
     (pin "2")
   )
-  (symbol (lib_id "mainboard-rescue:C-Device-mainboard-rescue") (at 41.91 101.6 270) (unit 1)
+  (symbol (lib_id "Device:C") (at 41.91 101.6 270) (unit 1)
     (in_bom yes) (on_board yes)
     (property "Reference" "C206" (id 0) (at 41.91 95.1992 90))
@@
     (pin "2")
   )
-  (symbol (lib_id "mainboard-rescue:C-Device-mainboard-rescue") (at 41.91 111.76 270) (unit 1)
+  (symbol (lib_id "Device:C") (at 41.91 111.76 270) (unit 1)
     (in_bom yes) (on_board yes)
     (property "Reference" "C207" (id 0) (at 41.91 105.3592 90))
@@
     (pin "2")
   )
-  (symbol (lib_id "mainboard-rescue:C-Device-mainboard-rescue") (at 41.91 121.92 270) (unit 1)
+  (symbol (lib_id "Device:C") (at 41.91 121.92 270) (unit 1)
     (in_bom yes) (on_board yes)
     (property "Reference" "C208" (id 0) (at 41.91 115.5192 90))
@@
     (pin "2")
   )
-  (symbol (lib_id "mainboard-rescue:C-Device-mainboard-rescue") (at 41.91 132.08 270) (unit 1)
+  (symbol (lib_id "Device:C") (at 41.91 132.08 270) (unit 1)
     (in_bom yes) (on_board yes)
     (property "Reference" "C209" (id 0) (at 41.91 125.6792 90))
@@
     (pin "2")
   )
-  (symbol (lib_id "mainboard-rescue:C-Device-mainboard-rescue") (at 154.94 63.5 0) (unit 1)
+  (symbol (lib_id "Device:C") (at 154.94 63.5 0) (unit 1)
     (in_bom yes) (on_board yes)
     (property "Reference" "C200" (id 0) (at 157.861 62.3316 0)
@@
     (pin "2")
   )
-  (symbol (lib_id "mainboard-rescue:C-Device-mainboard-rescue") (at 165.1 63.5 0) (unit 1)
+  (symbol (lib_id "Device:C") (at 165.1 63.5 0) (unit 1)
     (in_bom yes) (on_board yes)
     (property "Reference" "C201" (id 0) (at 168.021 62.3316 0)
