File: hardware/foras-promineo-revB-fm/Burn_Wires.kicad_sch (KiCad schematic)
At the start: 14 parts, among them Q20 IRF7404TRPBF, Q21 IRF7404TRPBF, Q4 DMN100-7-F, Q5 DMN100-7-F, Q6 SMMBT2222AWT1G, U16 PE014006

Commit message: fm sch changes
Parts:
- R25, R27, R28, R32, R33, R37, R38: symbol mainboard:RESISTOR0603 -> Device:R_US
