File: hardware/foras-promineo-revB-fm/Bus_Protection.kicad_sch (KiCad schematic)
At the start: 53 parts, among them Q11 MMDT2907AQ-7-F, Q12 BSS138DWQ-7, Q13 BSS138DWQ-7, Q15 MMDT5551-7-F, Q16 MMDT5551-7-F, Q17 FJV992FMTF, Q18 BSS138DWQ-7, Q19 BSS138DWQ-7, Q7 MMDT5551-7-F, Q8 MMDT5551-7-F

Commit message: fm sch changes
Parts:
- C40, C41, C42, C8: symbol mainboard-rescue:C-Device-mainboard-rescue -> Device:C
- R101, R104, R107, R108, R109, R48, R53, R60, R71, R72, R86, R87, R92, R97, R98, R99: symbol mainboard-rescue:R_US-Device-mainboard-rescue -> Device:R_US
- R61, R62, R66, R67, R82, R83, R84, R85: value 10K -> 10k; symbol mainboard-rescue:R_US-Device-mainboard-rescue -> Device:R_US
- R63, R64, R69, R70, R77, R78: value 1K -> 1k; symbol mainboard-rescue:R_US-Device-mainboard-rescue -> Device:R_US
- R68: value 4.7K -> 4.7k; symbol mainboard-rescue:R_US-Device-mainboard-rescue -> Device:R_US
- R73, R74, R93, R94: value 100K -> 100k; symbol mainboard-rescue:R_US-Device-mainboard-rescue -> Device:R_US
- R75, R76, R95, R96: value 200K -> 200k; symbol mainboard-rescue:R_US-Device-mainboard-rescue -> Device:R_US
