File: hardware/foras-promineo-revB-fm/Connectors.kicad_sch (KiCad schematic)
At the start: 6 parts, among them J1 503182-1852, J2 Conn_01x05, U8 MR25H40MDF

Commit message: fm sch changes
Parts:
- C30: symbol mainboard-rescue:C-Device-mainboard-rescue -> Device:C
- R50, R51: symbol mainboard-rescue:R_US-Device-mainboard-rescue -> Device:R_US
Changed lines of the file:
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@@
     (pin "9")
   )
-  (symbol (lib_id "mainboard-rescue:C-Device-mainboard-rescue") (at 80.01 115.57 0) (unit 1)
+  (symbol (lib_id "Device:C") (at 80.01 115.57 0) (unit 1)
     (in_bom yes) (on_board yes)
-    (property "Reference" "C30" (id 0) (at 81.534 112.649 0)
+    (property "Reference" "C30" (id 0) (at 84.074 113.919 0)
       (effects (font (size 1.778 1.778)) (justify left bottom))
     )
-    (property "Value" "0.1uF" (id 1) (at 81.534 117.729 0)
+    (property "Value" "0.1uF" (id 1) (at 84.074 117.729 0)
       (effects (font (size 1.778 1.778)) (justify left bottom))
     )
@@
     (pin "1")
   )
-  (symbol (lib_id "mainboard-rescue:R_US-Device-mainboard-rescue") (at 64.77 34.29 0) (mirror x) (unit 1)
+  (symbol (lib_id "Device:R_US") (at 64.77 34.29 0) (mirror x) (unit 1)
     (in_bom yes) (on_board yes)
     (property "Reference" "R51" (id 0) (at 62.23 31.75 0))
@@
     (pin "2")
   )
-  (symbol (lib_id "mainboard-rescue:R_US-Device-mainboard-rescue") (at 35.56 115.57 0) (mirror x) (unit 1)
+  (symbol (lib_id "Device:R_US") (at 35.56 115.57 0) (mirror x) (unit 1)
     (in_bom yes) (on_board yes)
     (property "Reference" "R50" (id 0) (at 33.02 113.03 0))
-    (property "Value" "10k" (id 1) (at 39.37 116.84 0))
+    (property "Value" "10k" (id 1) (at 33.02 115.57 0))
     (property "Footprint" "Resistor_SMD:R_0603_1608Metric" (id 2) (at 36.576 115.316 90)
       (effects (font (size 1.27 1.27)) hide)
