File: hardware/foras-promineo-revB-fm/IMU.kicad_sch (KiCad schematic)
At the start: 30 parts, among them U201 PCA9543APW,118, U204 IAM-20380, U205 MMC5983MA, U206 MXC6655XA, U207 IAM-20380, U208 MMC5983MA, U209 MXC6655XA

Commit message: fm sch changes
Parts:
- C217, C220, C221, C222, C223, C224, C225, C226, C227, C228, C229, C230, C231, C232, C233: symbol mainboard-rescue:C-Device-mainboard-rescue -> Device:C
- R229, R230, R231, R234, R235, R238, R239, R240: symbol mainboard-rescue:R_US-Device-mainboard-rescue -> Device:R_US
Changed lines of the file:
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@@
     (pin "1")
   )
-  (symbol (lib_id "mainboard-rescue:C-Device-mainboard-rescue") (at 31.75 158.75 0) (unit 1)
+  (symbol (lib_id "Device:C") (at 31.75 158.75 0) (unit 1)
     (in_bom yes) (on_board yes)
     (property "Reference" "C217" (id 0) (at 34.671 157.5816 0)
@@
     (pin "1")
   )
-  (symbol (lib_id "mainboard-rescue:R_US-Device-mainboard-rescue") (at 52.07 161.29 0) (unit 1)
+  (symbol (lib_id "Device:R_US") (at 52.07 161.29 0) (unit 1)
     (in_bom yes) (on_board yes)
     (property "Reference" "R240" (id 0) (at 53.7972 160.1216 0)
@@
     (pin "2")
   )
-  (symbol (lib_id "mainboard-rescue:R_US-Device-mainboard-rescue") (at 46.99 161.29 0) (unit 1)
+  (symbol (lib_id "Device:R_US") (at 46.99 161.29 0) (unit 1)
     (in_bom yes) (on_board yes)
     (property "Reference" "R239" (id 0) (at 40.64 160.02 0)
@@
     (pin "9")
   )
-  (symbol (lib_id "mainboard-rescue:R_US-Device-mainboard-rescue") (at 101.6 144.78 0) (unit 1)
+  (symbol (lib_id "Device:R_US") (at 101.6 144.78 0) (unit 1)
     (in_bom yes) (on_board yes)
     (property "Reference" "R229" (id 0) (at 103.3272 143.6116 0)
@@
     (pin "2")
   )
-  (symbol (lib_id "mainboard-rescue:R_US-Device-mainboard-rescue") (at 109.22 147.32 0) (unit 1)
+  (symbol (lib_id "Device:R_US") (at 109.22 147.32 0) (unit 1)
     (in_bom yes) (on_board yes)
     (property "Reference" "R230" (id 0) (at 110.9472 146.1516 0)
@@
     (pin "2")
   )
-  (symbol (lib_id "mainboard-rescue:R_US-Device-mainboard-rescue") (at 116.84 149.86 0) (unit 1)
+  (symbol (lib_id "Device:R_US") (at 116.84 149.86 0) (unit 1)
     (in_bom yes) (on_board yes)
     (property "Reference" "R231" (id 0) (at 118.5672 148.6916 0)
@@
     (pin "2")
   )
-  (symbol (lib_id "mainboard-rescue:R_US-Device-mainboard-rescue") (at 129.54 154.94 0) (unit 1)
+  (symbol (lib_id "Device:R_US") (at 129.54 154.94 0) (unit 1)
     (in_bom yes) (on_board yes)
     (property "Reference" "R234" (id 0) (at 131.2672 153.7716 0)
@@
     (pin "2")
   )
-  (symbol (lib_id "mainboard-rescue:R_US-Device-mainboard-rescue") (at 137.16 157.48 0) (unit 1)
+  (symbol (lib_id "Device:R_US") (at 137.16 157.48 0) (unit 1)
     (in_bom yes) (on_board yes)
     (property "Reference" "R235" (id 0) (at 138.8872 156.3116 0)
@@
     (pin "2")
   )
-  (symbol (lib_id "mainboard-rescue:R_US-Device-mainboard-rescue") (at 144.78 160.02 0) (unit 1)
+  (symbol (lib_id "Device:R_US") (at 144.78 160.02 0) (unit 1)
     (in_bom yes) (on_board yes)
     (property "Reference" "R238" (id 0) (at 146.5072 158.8516 0)
@@
     (pin "1")
   )
-  (symbol (lib_id "mainboard-rescue:C-Device-mainboard-rescue") (at 35.56 48.26 0) (unit 1)
+  (symbol (lib_id "Device:C") (at 35.56 48.26 0) (unit 1)
     (in_bom yes) (on_board yes)
     (property "Reference" "C224" (id 0) (at 38.481 47.0916 0)
@@
     (pin "1")
   )
-  (symbol (lib_id "mainboard-rescue:C-Device-mainboard-rescue") (at 24.13 48.26 0) (unit 1)
+  (symbol (lib_id "Device:C") (at 24.13 48.26 0) (unit 1)
     (in_bom yes) (on_board yes)
     (property "Reference" "C223" (id 0) (at 27.051 47.0916 0)
@@
     (pin "1")
   )
-  (symbol (lib_id "mainboard-rescue:C-Device-mainboard-rescue") (at 44.45 33.02 0) (unit 1)
+  (symbol (lib_id "Device:C") (at 44.45 33.02 0) (unit 1)
     (in_bom yes) (on_board yes)
     (property "Reference" "C220" (id 0) (at 47.371 31.8516 0)
@@
     (pin "1")
   )
-  (symbol (lib_id "mainboard-rescue:C-Device-mainboard-rescue") (at 45.72 52.07 0) (unit 1)
+  (symbol (lib_id "Device:C") (at 45.72 52.07 0) (unit 1)
     (in_bom yes) (on_board yes)
     (property "Reference" "C226" (id 0) (at 48.641 50.9016 0)
@@
     (pin "1")
   )
-  (symbol (lib_id "mainboard-rescue:C-Device-mainboard-rescue") (at 95.25 43.18 0) (unit 1)
+  (symbol (lib_id "Device:C") (at 95.25 43.18 0) (unit 1)
     (in_bom yes) (on_board yes)
     (property "Reference" "C221" (id 0) (at 98.171 42.0116 0)
@@
     (pin "1")
   )
-  (symbol (lib_id "mainboard-rescue:C-Device-mainboard-rescue") (at 105.41 49.53 0) (unit 1)
+  (symbol (lib_id "Device:C") (at 105.41 49.53 0) (unit 1)
     (in_bom yes) (on_board yes)
     (property "Reference" "C225" (id 0) (at 108.331 48.3616 0)
@@
     (pin "1")
   )
-  (symbol (lib_id "mainboard-rescue:C-Device-mainboard-rescue") (at 148.59 45.72 0) (unit 1)
+  (symbol (lib_id "Device:C") (at 148.59 45.72 0) (unit 1)
     (in_bom yes) (on_board yes)
     (property "Reference" "C222" (id 0) (at 151.511 44.5516 0)
@@
     (pin "1")
   )
-  (symbol (lib_id "mainboard-rescue:C-Device-mainboard-rescue") (at 34.29 106.68 0) (unit 1)
+  (symbol (lib_id "Device:C") (at 34.29 106.68 0) (unit 1)
     (in_bom yes) (on_board yes)
     (property "Reference" "C231" (id 0) (at 37.211 105.5116 0)
@@
     (pin "1")
   )
-  (symbol (lib_id "mainboard-rescue:C-Device-mainboard-rescue") (at 22.86 106.68 0) (unit 1)
+  (symbol (lib_id "Device:C") (at 22.86 106.68 0) (unit 1)
     (in_bom yes) (on_board yes)
     (property "Reference" "C230" (id 0) (at 25.781 105.5116 0)
@@
     (pin "1")
   )
-  (symbol (lib_id "mainboard-rescue:C-Device-mainboard-rescue") (at 43.18 91.44 0) (unit 1)
+  (symbol (lib_id "Device:C") (at 43.18 91.44 0) (unit 1)
     (in_bom yes) (on_board yes)
     (property "Reference" "C227" (id 0) (at 46.101 90.2716 0)
@@
     (pin "1")
   )
-  (symbol (lib_id "mainboard-rescue:C-Device-mainboard-rescue") (at 44.45 110.49 0) (unit 1)
+  (symbol (lib_id "Device:C") (at 44.45 110.49 0) (unit 1)
     (in_bom yes) (on_board yes)
     (property "Reference" "C233" (id 0) (at 47.371 109.3216 0)
@@
     (pin "1")
   )
-  (symbol (lib_id "mainboard-rescue:C-Device-mainboard-rescue") (at 93.98 101.6 0) (unit 1)
+  (symbol (lib_id "Device:C") (at 93.98 101.6 0) (unit 1)
     (in_bom yes) (on_board yes)
     (property "Reference" "C228" (id 0) (at 96.901 100.4316 0)
@@
     (pin "1")
   )
-  (symbol (lib_id "mainboard-rescue:C-Device-mainboard-rescue") (at 104.14 107.95 0) (unit 1)
+  (symbol (lib_id "Device:C") (at 104.14 107.95 0) (unit 1)
     (in_bom yes) (on_board yes)
     (property "Reference" "C232" (id 0) (at 107.061 106.7816 0)
@@
     (pin "1")
   )
-  (symbol (lib_id "mainboard-rescue:C-Device-mainboard-rescue") (at 147.32 104.14 0) (unit 1)
+  (symbol (lib_id "Device:C") (at 147.32 104.14 0) (unit 1)
     (in_bom yes) (on_board yes)
     (property "Reference" "C229" (id 0) (at 150.241 102.9716 0)
