File: hardware/foras-promineo-revB-fm/RF_and_GPS.kicad_sch (KiCad schematic)
At the start: 15 parts, among them J12 Amphenol_901-144, J5 Amphenol_901-144, J6 Amphenol_901-144, J7 Amphenol_901-144, U13 EP2W+, U14 S1216V8, U15 RFM9xBreakout, U20 RFM9xBreakout, U23 RFM98PW, U24 RFM98PW

Commit message: fm sch changes
Parts:
- removed J6: Amphenol_901-144, Connector_Coaxial:SMA_Amphenol_901-144_Vertical, symbol mainboard-rescue:Conn_Coaxial-Connector-mainboard-rescue
- removed U13: EP2W+, mainboard:QFN32-5X5MM, symbol mainboard:EP2W+
- C44, C46: symbol mainboard-rescue:C_Small-Device-mainboard-rescue -> Device:C_Small
- R24: value 10K -> 10k; symbol mainboard:10KOHM-1_10W-1%(0603)0603 -> Device:R_US
- R43, R5: symbol mainboard:10KOHM-1_10W-1%(0603)0603 -> Device:R_US
Connections:
- net VCC_RF1 is gone; now on net 3.3V: C44.2, U20.13 (3V3), U23.5 (VCC)
- net VCC_RF2 is gone; now on net 3.3V: C46.2, U15.13 (3V3), U24.5 (VCC)
- net RF_IN: now also J5.1 (In)
