File: hardware/foras-promineo-revB-fm/Power.kicad_sch (KiCad schematic)
At the start: 45 parts, among them Q1 DMN100-7-F, Q2 MMDT5551-7-F, Q22 IRF7404TRPBF, Q3 MMDT5551-7-F, U17 BQ25883RGER, U4 ADM1176-1ARMZ-R7, U5 TPS54226PWPRPWP14_2P31X2P46-L

Commit message: friday updates
Connections:
- net VBATT renamed VCHRG
Other:
- note added: "(power TO bus)"
Changed lines of the file:
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@@
     (stroke (width 0) (type default) (color 0 0 0 0))
+  )
+  (text "(power TO bus)" (at 130.81 88.9 0)
+    (effects (font (size 1.27 1.27)) (justify left bottom))
   )
   (text "Value is convenient,\nnot necessary. \n10K-80K would\nalso work for R29"
@@
     )
   )
-  (global_label "VBATT" (shape bidirectional) (at 115.57 88.9 180) (fields_autoplaced)
-    (effects (font (size 1.27 1.27)) (justify right))
-    (property "Intersheet References" "${INTERSHEET_REFS}" (id 0) (at 0 0 0)
-      (effects (font (size 1.27 1.27)) hide)
-    )
-  )
   (global_label "GND" (shape bidirectional) (at 180.34 97.79 180) (fields_autoplaced)
     (effects (font (size 0.254 0.254)) (justify right))
@@
     )
   )
+  (global_label "VCHRG" (shape input) (at 115.57 88.9 180) (fields_autoplaced)
+    (effects (font (size 1.27 1.27)) (justify right))
+    (property "Intersheet References" "${INTERSHEET_REFS}" (id 0) (at 107.0168 88.9794 0)
+      (effects (font (size 1.27 1.27)) (justify right) hide)
+    )
+  )

Commit message: fm sch changes
Parts:
- removed JP6, JP7: Jumper_3_Bridged12, mainboard:SolderJumper-3_P1.3mm_Bridged12_RoundedPad1.0x1.5mm, symbol mainboard-rescue:Jumper_3_Bridged12-Jumper-mainboard-rescue
- C17, C18: symbol mainboard:22UF-0805-6.3V-20% -> Device:C
- C19, C20: symbol mainboard:22UF-1210-16V-20% -> Device:C
- C21, C27: symbol mainboard:1.0UF-0603-16V-10% -> Device:C
- C26: symbol mainboard:3.3NF-0603-100V-10% -> Device:C
- C32, C34, C36, C37, C38, C39: symbol mainboard-rescue:C-Device-mainboard-rescue -> Device:C
- C33, C35, C6: symbol mainboard-rescue:C_Small-Device-mainboard-rescue -> Device:C_Small
- L2, L4: symbol mainboard-rescue:L-Device-mainboard-rescue -> Device:L
- Q2: Manufacturer_Name (none) -> ON Semiconductor; Manufacturer_Part_Number (none) -> MBT2222ADW1T1G; Proto (none) -> MBT2222ADW1T1G
- R110: value 20K -> 20k; symbol mainboard-rescue:R_US-Device-mainboard-rescue -> Device:R_US
- R13: value 73.2K -> 73.2k; symbol mainboard:R-US_R0603 -> Device:R_US
- R14: value 22.1K -> 22.1k; symbol mainboard:R-US_R0603 -> Device:R_US
- R15: value 100K -> 100k; symbol mainboard:R-US_R0603 -> Device:R_US
- R21: value 10K -> 10k; symbol mainboard:R-US_R0603 -> Device:R_US
- R22: value 4.7K -> 4.7k; symbol mainboard:R-US_R0603 -> Device:R_US
- R23: value 3.3K -> 3.3k; symbol mainboard:R-US_R0603 -> Device:R_US
- R26: value 1K -> 1k; symbol mainboard-rescue:R_US-Device-mainboard-rescue -> Device:R_US
- R29: value 73.2K -> 73.2k; symbol mainboard-rescue:R_US-Device-mainboard-rescue -> Device:R_US
- R30, R49: value 100K -> 100k; symbol mainboard-rescue:R_US-Device-mainboard-rescue -> Device:R_US
- R34: value 5.23K -> 5.23k; symbol mainboard-rescue:R_US-Device-mainboard-rescue -> Device:R_US
- R35: value 30.1K -> 30.1k; symbol mainboard-rescue:R_US-Device-mainboard-rescue -> Device:R_US
- R36: value 3.16K -> 3.16k; symbol mainboard-rescue:R_US-Device-mainboard-rescue -> Device:R_US
- R46, R52: value 10K -> 10k; symbol mainboard-rescue:R_US-Device-mainboard-rescue -> Device:R_US
- R47: value 200K -> 200k; symbol mainboard-rescue:R_US-Device-mainboard-rescue -> Device:R_US
- R8: symbol mainboard:R-US_R2512 -> Device:R_US
Other:
- note removed: "Radio VDD Select"
- note removed: "remove these jumpers? i dont think we need this."

Commit message: fm layout work
Changed lines of the file:
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@@
-    (stroke (width 0) (type default) (color 0 0 0 0))
-  )
-  (wire (pts (xy 252.73 88.9) (xy 252.73 86.36))
     (stroke (width 0) (type default) (color 0 0 0 0))
   )
@@
   )
   (wire (pts (xy 123.19 173.99) (xy 135.89 173.99))
-    (stroke (width 0) (type default) (color 0 0 0 0))
-  )
-  (wire (pts (xy 252.73 86.36) (xy 255.27 86.36))
     (stroke (width 0) (type default) (color 0 0 0 0))
   )
@@
   )
   (global_label "VBUS_RESET" (shape input) (at 179.07 154.94 0) (fields_autoplaced)
-    (effects (font (size 1.27 1.27)) (justify left))
-    (property "Intersheet References" "${INTERSHEET_REFS}" (id 0) (at 0 0 0)
-      (effects (font (size 1.27 1.27)) hide)
-    )
-  )
-  (global_label "VBATT_RET" (shape bidirectional) (at 255.27 86.36 0) (fields_autoplaced)
     (effects (font (size 1.27 1.27)) (justify left))
     (property "Intersheet References" "${INTERSHEET_REFS}" (id 0) (at 0 0 0)
@@
     (pin "2")
   )
-  (symbol (lib_id "mainboard-rescue:GNDREF-power-mainboard-rescue") (at 252.73 88.9 0) (unit 1)
-    (in_bom yes) (on_board yes)
-    (property "Reference" "#PWR0106" (id 0) (at 252.73 95.25 0)
-      (effects (font (size 1.27 1.27)) hide)
-    )
-    (property "Value" "GNDREF" (id 1) (at 252.857 93.2942 0))
-    (property "Footprint" "" (id 2) (at 252.73 88.9 0)
-      (effects (font (size 1.27 1.27)) hide)
-    )
-    (property "Datasheet" "" (id 3) (at 252.73 88.9 0)
-      (effects (font (size 1.27 1.27)) hide)
-    )
-    (pin "1")
-  )
   (symbol (lib_id "mainboard-rescue:GNDREF-power-mainboard-rescue") (at 204.47 152.4 0) (unit 1)
