File: hardware/foras-promineo-revB-fm/Avionics.kicad_sch (KiCad schematic)
At the start: 32 parts, among them SW1 KMR231NG LFS, U1 MAX706RESA, U2 ATSAMD51N20A-AUT, Y1 32.768kHz

Commit message: added charge current monitor
Connections:
- net ~{CHRG_SHDN}: now reaches U2.69 (PB21)
Changed lines of the file:
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@@
+    )
+  )
+  (global_label "~{CHRG_SHDN}" (shape output) (at 90.17 168.91 180) (fields_autoplaced)
+    (effects (font (size 1.27 1.27)) (justify right))
+    (property "Intersheet References" "${INTERSHEET_REFS}" (id 0) (at 76.5972 168.8306 0)
+      (effects (font (size 1.27 1.27)) (justify right) hide)
     )
   )

Commit message: updating FM
Connections:
- net NeoPixel_Out: now reaches D1.2 (DOUT)
- no-connect marks 13 -> 12
Other:
- moved on the sheet: C5
Changed lines of the file:
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@@
   (no_connect (at 90.17 171.45))
   (no_connect (at 90.17 181.61))
-  (no_connect (at 46.99 99.06))
   (no_connect (at 146.05 97.79))
   (no_connect (at 146.05 95.25))
@@
     (stroke (width 0) (type default) (color 0 0 0 0))
   )
-  (wire (pts (xy 40.64 106.68) (xy 40.64 104.14))
+  (wire (pts (xy 29.21 106.68) (xy 29.21 104.14))
     (stroke (width 0) (type default) (color 0 0 0 0))
   )
@@
     (stroke (width 0) (type default) (color 0 0 0 0))
   )
-  (wire (pts (xy 40.64 106.68) (xy 54.61 106.68))
+  (wire (pts (xy 29.21 106.68) (xy 54.61 106.68))
     (stroke (width 0) (type default) (color 0 0 0 0))
   )
@@
     (stroke (width 0) (type default) (color 0 0 0 0))
   )
-  (wire (pts (xy 40.64 91.44) (xy 54.61 91.44))
+  (wire (pts (xy 29.21 91.44) (xy 54.61 91.44))
     (stroke (width 0) (type default) (color 0 0 0 0))
   )
@@
     (stroke (width 0) (type default) (color 0 0 0 0))
   )
-  (wire (pts (xy 40.64 96.52) (xy 40.64 91.44))
+  (wire (pts (xy 29.21 96.52) (xy 29.21 91.44))
     (stroke (width 0) (type default) (color 0 0 0 0))
   )
@@
     (property "Intersheet References" "${INTERSHEET_REFS}" (id 0) (at 0 0 0)
       (effects (font (size 1.27 1.27)) hide)
+    )
+  )
+  (global_label "NeoPixel_Out" (shape input) (at 46.99 99.06 180) (fields_autoplaced)
+    (effects (font (size 1.27 1.27)) (justify right))
+    (property "Intersheet References" "${INTERSHEET_REFS}" (id 0) (at 32.2682 98.9806 0)
+      (effects (font (size 1.27 1.27)) (justify right) hide)
     )
   )
@@
     (pin "1")
   )
-  (symbol (lib_id "mainboard-rescue:C-Device-mainboard-rescue") (at 40.64 100.33 0) (unit 1)
-    (in_bom yes) (on_board yes)
-    (property "Reference" "C5" (id 0) (at 36.83 96.52 0)
+  (symbol (lib_id "mainboard-rescue:C-Device-mainboard-rescue") (at 29.21 100.33 0) (unit 1)
+    (in_bom yes) (on_board yes)
+    (property "Reference" "C5" (id 0) (at 25.4 96.52 0)
       (effects (font (size 1.4986 1.4986)) (justify right top))
     )
-    (property "Value" "0.1uF" (id 1) (at 36.83 99.06 0)
+    (property "Value" "0.1uF" (id 1) (at 25.4 99.06 0)
       (effects (font (size 1.4986 1.4986)) (justify right top))
     )
-    (property "Footprint" "Capacitor_SMD:C_0603_1608Metric" (id 2) (at 40.64 100.33 0)
-      (effects (font (size 1.27 1.27)) hide)
-    )
-    (property "Datasheet" "" (id 3) (at 40.64 100.33 0)
-      (effects (font (size 1.27 1.27)) hide)
-    )
-    (property "Description" "" (id 4) (at 40.64 100.33 0)
-      (effects (font (size 1.27 1.27)) hide)
-    )
+    (property "Footprint" "Capacitor_SMD:C_0603_1608Metric" (id 2) (at 29.21 100.33 0)
+      (effects (font (size 1.27 1.27)) hide)
+    )
+    (property "Datasheet" "" (id 3) (at 29.21 100.33 0)
+      (effects (font (size 1.27 1.27)) hide)
+    )
+    (property "Description" "" (id 4) (at 29.21 100.33 0)
+      (effects (font (size 1.27 1.27)) hide)
+    )

Commit message: friday updates
Parts:
- added R6: 100k, Resistor_SMD:R_0603_1608Metric, symbol Device:R_US
Connections:
- net 3.3V: now also R6.1
- net AIN7: now reaches U2.20 (PA07)
- net MUX_S0: now reaches U2.72 (PA22)
- net ~{SELF_TEST}: now reaches U2.78 (PB22)
- net ~{SELF_TEST}: now also R6.2
- net ~{USB_EN}: now reaches U2.79 (PB23)
- net MUX_S1: now reaches U2.80 (PB24)
- net MUX_S2: now reaches U2.81 (PB25)
- net MUX_S3: now reaches U2.95 (PB30)
- net ~{MUX_EN}: now reaches U2.96 (PB31)
- net PC00 renamed AIN10
- net PC01 renamed AIN11
- net PC02 renamed AIN4
- no-connect marks 12 -> 5
Changed lines of the file:
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@@
   (junction (at 161.29 27.94) (diameter 0) (color 0 0 0 0)
   )
+  (junction (at 60.96 171.45) (diameter 0) (color 0 0 0 0)
+  )
   (junction (at 46.99 45.72) (diameter 0) (color 0 0 0 0)
   )
@@
   (junction (at 168.91 35.56) (diameter 0) (color 0 0 0 0)
   )
-  (no_connect (at 90.17 179.07))
   (no_connect (at 220.98 62.23))
   (no_connect (at 146.05 100.33))
   (no_connect (at 146.05 102.87))
-  (no_connect (at 90.17 184.15))
-  (no_connect (at 90.17 173.99))
-  (no_connect (at 90.17 176.53))
-  (no_connect (at 90.17 171.45))
-  (no_connect (at 90.17 181.61))
   (no_connect (at 146.05 97.79))
   (no_connect (at 146.05 95.25))
-  (no_connect (at 90.17 63.5))
   (wire (pts (xy 63.5 27.94) (xy 73.66 27.94))
     (stroke (width 0) (type default) (color 0 0 0 0))
@@
     (stroke (width 0) (type default) (color 0 0 0 0))
   )
+  (wire (pts (xy 60.96 171.45) (xy 90.17 171.45))
+    (stroke (width 0) (type default) (color 0 0 0 0))
+  )
   (wire (pts (xy 44.45 45.72) (xy 46.99 45.72))
     (stroke (width 0) (type default) (color 0 0 0 0))
@@
   )
   (polyline (pts (xy 101.6 86.36) (xy 102.87 86.36))
+    (stroke (width 0) (type default) (color 0 0 0 0))
+  )
+  (wire (pts (xy 44.45 171.45) (xy 60.96 171.45))
     (stroke (width 0) (type default) (color 0 0 0 0))
   )
@@
     (effects (font (size 1.4986 1.4986)) (justify left bottom))
   )
+  (global_label "AIN7" (shape bidirectional) (at 90.17 63.5 180) (fields_autoplaced)
+    (effects (font (size 1.27 1.27)) (justify right))
+    (property "Intersheet References" "${INTERSHEET_REFS}" (id 0) (at 83.6125 63.4206 0)
+      (effects (font (size 1.27 1.27)) (justify right) hide)
+    )
+  )
   (global_label "ENAB_BURN1" (shape bidirectional) (at 146.05 107.95 0) (fields_autoplaced)
     (effects (font (size 0.9906 0.9906)) (justify left))
@@
     )
   )
+  (global_label "MUX_S2" (shape input) (at 90.17 179.07 180) (fields_autoplaced)
+    (effects (font (size 1.27 1.27)) (justify right))
+    (property "Intersheet References" "${INTERSHEET_REFS}" (id 0) (at 80.4677 178.9906 0)
+      (effects (font (size 1.27 1.27)) (justify right) hide)
+    )
+  )
   (global_label "SWCLK" (shape bidirectional) (at 82.55 33.02 180) (fields_autoplaced)
     (effects (font (size 1.27 1.27)) (justify right))
@@
     )
   )
+  (global_label "~{USB_EN}" (shape output) (at 90.17 173.99 180) (fields_autoplaced)
+    (effects (font (size 1.27 1.27)) (justify right))
+    (property "Intersheet References" "${INTERSHEET_REFS}" (id 0) (at 80.5887 173.9106 0)
+      (effects (font (size 1.27 1.27)) (justify right) hide)
+    )
+  )
   (global_label "RF2_CS" (shape bidirectional) (at 90.17 138.43 180) (fields_autoplaced)
     (effects (font (size 1.27 1.27)) (justify right))
@@
     )
   )
-  (global_label "PC01" (shape input) (at 146.05 54.61 0) (fields_autoplaced)
+  (global_label "AIN11" (shape input) (at 146.05 54.61 0) (fields_autoplaced)
     (effects (font (size 1.27 1.27)) (justify left))
-    (property "Intersheet References" "${INTERSHEET_REFS}" (id 0) (at 0 0 0)
-      (effects (font (size 1.27 1.27)) hide)
+    (property "Intersheet References" "${INTERSHEET_REFS}" (id 0) (at 153.8171 54.5306 0)
+      (effects (font (size 1.27 1.27)) (justify left) hide)
     )
   )
@@
     (property "Intersheet References" "${INTERSHEET_REFS}" (id 0) (at 0 0 0)
       (effects (font (size 1.27 1.27)) hide)
+    )
+  )
+  (global_label "~{MUX_EN}" (shape input) (at 90.17 184.15 180) (fields_autoplaced)
+    (effects (font (size 1.27 1.27)) (justify right))
+    (property "Intersheet References" "${INTERSHEET_REFS}" (id 0) (at 80.4072 184.0706 0)
+      (effects (font (size 1.27 1.27)) (justify right) hide)
     )
   )
@@
     )
   )
+  (global_label "MUX_S1" (shape input) (at 90.17 176.53 180) (fields_autoplaced)
+    (effects (font (size 1.27 1.27)) (justify right))
+    (property "Intersheet References" "${INTERSHEET_REFS}" (id 0) (at 80.4677 176.4506 0)
+      (effects (font (size 1.27 1.27)) (justify right) hide)
+    )
+  )
   (global_label "EN_PAYLOAD" (shape bidirectional) (at 90.17 163.83 180) (fields_autoplaced)
     (effects (font (size 0.9906 0.9906)) (justify right))
@@
     )
   )
+  (global_label "MUX_S3" (shape input) (at 90.17 181.61 180) (fields_autoplaced)
+    (effects (font (size 1.27 1.27)) (justify right))
+    (property "Intersheet References" "${INTERSHEET_REFS}" (id 0) (at 80.4677 181.5306 0)
+      (effects (font (size 1.27 1.27)) (justify right) hide)
+    )
+  )
   (global_label "RF1_RST" (shape bidirectional) (at 90.17 115.57 180) (fields_autoplaced)
     (effects (font (size 1.27 1.27)) (justify right))
@@
     )
   )
-  (global_label "PC00" (shape input) (at 146.05 52.07 0) (fields_autoplaced)
+  (global_label "MUX_S0" (shape input) (at 90.17 101.6 180) (fields_autoplaced)
+    (effects (font (size 1.27 1.27)) (justify right))
+    (property "Intersheet References" "${INTERSHEET_REFS}" (id 0) (at 80.4677 101.5206 0)
+      (effects (font (size 1.27 1.27)) (justify right) hide)
+    )
+  )
+  (global_label "AIN10" (shape input) (at 146.05 52.07 0) (fields_autoplaced)
     (effects (font (size 1.27 1.27)) (justify left))
-    (property "Intersheet References" "${INTERSHEET_REFS}" (id 0) (at 0 0 0)
-      (effects (font (size 1.27 1.27)) hide)
+    (property "Intersheet References" "${INTERSHEET_REFS}" (id 0) (at 153.8171 51.9906 0)
+      (effects (font (size 1.27 1.27)) (justify left) hide)
     )
   )
@@
     )
   )
-  (global_label "PC02" (shape input) (at 146.05 57.15 0) (fields_autoplaced)
+  (global_label "AIN4" (shape input) (at 146.05 57.15 0) (fields_autoplaced)
     (effects (font (size 1.27 1.27)) (justify left))
-    (property "Intersheet References" "${INTERSHEET_REFS}" (id 0) (at 0 0 0)
-      (effects (font (size 1.27 1.27)) hide)
+    (property "Intersheet References" "${INTERSHEET_REFS}" (id 0) (at 152.6075 57.0706 0)
+      (effects (font (size 1.27 1.27)) (justify left) hide)
     )
   )
@@
     (property "Intersheet References" "${INTERSHEET_REFS}" (id 0) (at 0 0 0)
       (effects (font (size 1.27 1.27)) hide)
+    )
+  )
+  (global_label "~{SELF_TEST}" (shape input) (at 44.45 171.45 180) (fields_autoplaced)
+    (effects (font (size 1.27 1.27)) (justify right))
+    (property "Intersheet References" "${INTERSHEET_REFS}" (id 0) (at 32.3891 171.3706 0)
+      (effects (font (size 1.27 1.27)) (justify right) hide)
     )
   )
@@
     (pin "2")
   )
+  (symbol (lib_id "Device:R_US") (at 60.96 167.64 0) (unit 1)
+    (in_bom yes) (on_board yes) (fields_autoplaced)
+    (property "Reference" "R6" (id 0) (at 63.5 166.3699 0)
+      (effects (font (size 1.27 1.27)) (justify left))
+    )
+    (property "Value" "100k" (id 1) (at 63.5 168.9099 0)
+      (effects (font (size 1.27 1.27)) (justify left))
+    )
+    (property "Footprint" "Resistor_SMD:R_0603_1608Metric" (id 2) (at 61.976 167.894 90)
+      (effects (font (size 1.27 1.27)) hide)
+    )
+    (property "Datasheet" "~" (id 3) (at 60.96 167.64 0)
+      (effects (font (size 1.27 1.27)) hide)
+    )
+    (pin "1")
+    (pin "2")
+  )
+  (symbol (lib_id "mainboard:3.3V") (at 60.96 163.83 0) (mirror y) (unit 1)
+    (in_bom yes) (on_board yes)
+    (property "Reference" "#SUPPLY0111" (id 0) (at 60.96 163.83 0)
+      (effects (font (size 1.27 1.27)) hide)
+    )
+    (property "Value" "3.3V" (id 1) (at 63.5 160.02 0)
+      (effects (font (size 1.4986 1.4986)) (justify left bottom))
+    )
+    (property "Footprint" "" (id 2) (at 60.96 163.83 0)
+      (effects (font (size 1.27 1.27)) hide)
+    )
+    (property "Datasheet" "" (id 3) (at 60.96 163.83 0)
+      (effects (font (size 1.27 1.27)) hide)
+    )
+    (pin "1")
+  )
 )

Commit message: fm sch changes
Parts:
- C1, C10, C11, C12, C13, C14, C15, C16, C2, C218, C219, C234, C251, C252, C253, C3, C4, C5: symbol mainboard-rescue:C-Device-mainboard-rescue -> Device:C
- L1: symbol mainboard:INDUCTOR-Adafruit_Feather_M4_Express-eagle-import-lab64_SAM32-rescue-SAMD-10-rescue-SAM32-rescue -> Device:L
- R1: value 316K -> 316k; symbol mainboard-rescue:R_US-Device-mainboard-rescue -> Device:R_US
- R2: value 110K -> 110k; symbol mainboard-rescue:R_US-Device-mainboard-rescue -> Device:R_US
- R3, R4, R44, R45: value 10K -> 10k; symbol mainboard-rescue:R_US-Device-mainboard-rescue -> Device:R_US
- R42: symbol mainboard-rescue:R_US-Device-mainboard-rescue -> Device:R_US
- R7: symbol mainboard:R-US_R0603 -> Device:R_US
- Y1: symbol mainboard-rescue:Crystal-Device-mainboard-rescue -> Device:Crystal
Connections:
- net GND: no longer R7.1
- net WDT_WDI: no longer R7.2
- net at C12.2, C14.1, U2.89 (VDDCORE): now also L1.2; no longer L1.1
- net at U2.91 (VSW): now also L1.1; no longer L1.2
Other:
- note added: "CHECK L1"

Commit message: fm layout work
Parts:
- L1: Flight MGFL2012F100MT-LF -> (none); Manufacturer_Name MicroGate -> (none); Manufacturer_Part_Number MGFL2012F100MT-LF -> (none); Proto MGFL2012F100MT-LF -> (none)
Connections:
- net GND: now also R7.2
- net WDT_WDI: now also R7.1
Other:
- note removed: "CHECK L1"
- note removed: "switch output caps"
- moved on the sheet: R7
Changed lines of the file:
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@@
   (junction (at 58.42 67.31) (diameter 0) (color 0 0 0 0)
+  )
+  (junction (at 73.66 104.14) (diameter 0) (color 0 0 0 0)
   )
   (junction (at 146.05 27.94) (diameter 0) (color 0 0 0 0)
@@
     (stroke (width 0) (type default) (color 0 0 0 0))
   )
+  (wire (pts (xy 73.66 113.03) (xy 73.66 114.3))
+    (stroke (width 0) (type default) (color 0 0 0 0))
+  )
   (wire (pts (xy 146.05 27.94) (xy 154.94 27.94))
     (stroke (width 0) (type default) (color 0 0 0 0))
@@
     (stroke (width 0) (type default) (color 0 0 0 0))
   )
-  (wire (pts (xy 71.12 104.14) (xy 90.17 104.14))
+  (wire (pts (xy 71.12 104.14) (xy 73.66 104.14))
     (stroke (width 0) (type default) (color 0 0 0 0))
   )
@@
     (stroke (width 0) (type default) (color 0 0 0 0))
   )
+  (wire (pts (xy 73.66 104.14) (xy 73.66 105.41))
+    (stroke (width 0) (type default) (color 0 0 0 0))
+  )
   (wire (pts (xy 60.96 171.45) (xy 90.17 171.45))
     (stroke (width 0) (type default) (color 0 0 0 0))
@@
     (stroke (width 0) (type default) (color 0 0 0 0))
   )
+  (wire (pts (xy 73.66 104.14) (xy 90.17 104.14))
+    (stroke (width 0) (type default) (color 0 0 0 0))
+  )
   (wire (pts (xy 196.85 27.94) (xy 204.47 27.94))
     (stroke (width 0) (type default) (color 0 0 0 0))
@@
   )
   (text "sercom m7 pad[1]" (at 160.02 78.74 0)
-    (effects (font (size 1.27 1.27)) (justify left bottom))
-  )
-  (text "CHECK L1" (at 144.78 49.53 0)
     (effects (font (size 1.27 1.27)) (justify left bottom))
   )
@@
   (text "sercom m6 pad[0]" (at 160.02 85.09 0)
     (effects (font (size 1.27 1.27)) (justify left bottom))
-  )
-  (text "switch output caps" (at 158.75 41.91 0)
-    (effects (font (size 1.4986 1.4986)) (justify left bottom))
   )
   (text "TCK\nTMS" (at 102.87 30.48 0)
@@
       (effects (font (size 1.27 1.27)) hide)
     )
-    (property "Datasheet" "" (id 3) (at 151.13 43.18 0)
-      (effects (font (size 1.27 1.27)) hide)
-    )
-    (property "Description" "10uH Unshielded 0805" (id 4) (at 151.13 43.18 0)
-      (effects (font (size 1.27 1.27)) hide)
-    )
-    (property "Flight" "MGFL2012F100MT-LF" (id 5) (at 151.13 43.18 0)
-      (effects (font (size 1.27 1.27)) hide)
-    )
-    (property "Manufacturer_Name" "MicroGate" (id 6) (at 151.13 43.18 0)
-      (effects (font (size 1.27 1.27)) hide)
-    )
-    (property "Manufacturer_Part_Number" "MGFL2012F100MT-LF" (id 7) (at 149.86 43.18 0)
-      (effects (font (size 1.27 1.27)) hide)
-    )
-    (property "Proto" "MGFL2012F100MT-LF" (id 8) (at 151.13 43.18 0)
+    (property "Datasheet" "BCL322520RT-100M-D" (id 3) (at 151.13 43.18 0)
       (effects (font (size 1.27 1.27)) hide)
     )
@@
     (pin "1")
   )
-  (symbol (lib_id "Device:R_US") (at 73.66 109.22 270) (mirror x) (unit 1)
-    (in_bom yes) (on_board yes)
-    (property "Reference" "R7" (id 0) (at 67.31 108.1786 90)
+  (symbol (lib_id "Device:R_US") (at 73.66 109.22 0) (mirror y) (unit 1)
+    (in_bom yes) (on_board yes)
+    (property "Reference" "R7" (id 0) (at 71.12 110.2106 0)
       (effects (font (size 1.4986 1.4986)) (justify left bottom))
     )
-    (property "Value" "10k" (id 1) (at 67.31 110.998 90)
+    (property "Value" "10k" (id 1) (at 71.12 113.03 0)
       (effects (font (size 1.4986 1.4986)) (justify left bottom))
     )
@@
       (effects (font (size 1.27 1.27)) hide)
     )
-    (property "Description" "" (id 4) (at 69.85 108.1786 0)
-      (effects (font (size 1.27 1.27)) hide)
-    )
+    (property "Description" "" (id 4) (at 72.6186 113.03 0)
+      (effects (font (size 1.27 1.27)) hide)
+    )

Commit message: more fm layout
Connections:
- net ~{USB_EN}: no longer names the net of U2.79 (PB23)
Changed lines of the file:
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@@
-    )
-  )
-  (global_label "~{USB_EN}" (shape output) (at 90.17 173.99 180) (fields_autoplaced)
-    (effects (font (size 1.27 1.27)) (justify right))
-    (property "Intersheet References" "${INTERSHEET_REFS}" (id 0) (at 80.5887 173.9106 0)
-      (effects (font (size 1.27 1.27)) (justify right) hide)
     )
   )
