File: hardware/foras-promineo-revB-fm/SLI-Backplane-Blank-Card-KiCad.kicad_sch (KiCad schematic)
At the start: 25 parts, among them J201 TSM-102-01-L-SV-P-TR, P1 Card Edge for HSEC8-160-01-S-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, Q205 MMBT4401-7-F, Q206 IRF7458, Q207 IRF7404, Q208 IRF7458, Q211 IRF7404, Q212 IRF7404, Q213 IRF7404, Q220 IRF7404

Commit message: more testing
Other:
- note added: "fix this ckt"
Changed lines of the file:
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@@
+    (effects (font (size 1.27 1.27)) (justify left bottom))
+  )
+  (text "fix this ckt" (at 260.35 201.93 0)
     (effects (font (size 1.27 1.27)) (justify left bottom))
   )

Commit message: updating FM
Parts:
- Q205: symbol mainboard-rescue:Q_NPN_BCE-Device-mainboard-rescue -> mainboard-rescue:Q_NPN_BEC-Device-mainboard-rescue
Connections:
- net GNDREF: now also Q205.2 (E); no longer Q205.3 (E)
- net at Q207.4 (G), R216.2: now also Q205.3 (C); no longer Q205.2 (C)
- net BP_LED_LATCH renamed NeoPixel_Out
Other:
- note added: "irridum OnOff (high pulls low)"
- note added: "irridum pw sw en"
- note added: "payload RST"
- note added: "payload SERVO_PWR_CTRL"
- note added: "payload pw sw en"
- note added: "pico pw sw en"
- note added: "startracker RST"
- note added: "startracker pw sw en"
- note removed: "currently unused, going to go somehwere eventually?"
- note removed: "enable irridium"
- note removed: "enable openLST"
Changed lines of the file:
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@@
+    (stroke (width 0) (type default) (color 0 0 0 0))
+  )
+  (polyline (pts (xy 49.53 240.03) (xy 49.53 240.03))
     (stroke (width 0) (type default) (color 0 0 0 0))
   )
@@
     (stroke (width 0) (type default) (color 0 0 0 0))
   )
+  (polyline (pts (xy 41.91 237.49) (xy 49.53 237.49))
+    (stroke (width 0) (type default) (color 0 0 0 0))
+  )
   (wire (pts (xy 91.44 67.31) (xy 69.85 67.31))
     (stroke (width 0) (type default) (color 0 0 0 0))
@@
     (stroke (width 0) (type default) (color 0 0 0 0))
   )
+  (polyline (pts (xy 49.53 237.49) (xy 49.53 237.49))
+    (stroke (width 0) (type default) (color 0 0 0 0))
+  )
   (wire (pts (xy 57.15 62.23) (xy 35.56 62.23))
     (stroke (width 0) (type default) (color 0 0 0 0))
@@
     (stroke (width 0) (type default) (color 0 0 0 0))
   )
+  (polyline (pts (xy 41.91 234.95) (xy 49.53 234.95))
+    (stroke (width 0) (type default) (color 0 0 0 0))
+  )
   (wire (pts (xy 142.24 148.59) (xy 118.11 148.59))
     (stroke (width 0) (type default) (color 0 0 0 0))
@@
     (stroke (width 0) (type default) (color 0 0 0 0))
   )
+  (polyline (pts (xy 41.91 242.57) (xy 49.53 242.57))
+    (stroke (width 0) (type default) (color 0 0 0 0))
+  )
   (wire (pts (xy 189.23 49.53) (xy 180.34 49.53))
     (stroke (width 0) (type default) (color 0 0 0 0))
@@
     (stroke (width 0) (type default) (color 0 0 0 0))
   )
+  (polyline (pts (xy 41.91 245.11) (xy 49.53 245.11))
+    (stroke (width 0) (type default) (color 0 0 0 0))
+  )
   (wire (pts (xy 57.15 153.67) (xy 35.56 153.67))
     (stroke (width 0) (type default) (color 0 0 0 0))
@@
   )
   (wire (pts (xy 57.15 54.61) (xy 35.56 54.61))
+    (stroke (width 0) (type default) (color 0 0 0 0))
+  )
+  (polyline (pts (xy 41.91 240.03) (xy 49.53 240.03))
     (stroke (width 0) (type default) (color 0 0 0 0))
   )
@@
     (stroke (width 0) (type default) (color 0 0 0 0))
   )
+  (polyline (pts (xy 41.91 247.65) (xy 49.53 247.65))
+    (stroke (width 0) (type default) (color 0 0 0 0))
+  )
   (wire (pts (xy 57.15 110.49) (xy 35.56 110.49))
     (stroke (width 0) (type default) (color 0 0 0 0))
@@
     (stroke (width 0) (type default) (color 0 0 0 0))
   )
+  (polyline (pts (xy 41.91 232.41) (xy 49.53 232.41))
+    (stroke (width 0) (type default) (color 0 0 0 0))
+  )
   (polyline (pts (xy 38.1 214.63) (xy 40.64 214.63))
     (stroke (width 0) (type default) (color 0 0 0 0))
@@
     (stroke (width 0) (type default) (color 0 0 0 0))
   )
+  (polyline (pts (xy 41.91 250.19) (xy 49.53 250.19))
+    (stroke (width 0) (type default) (color 0 0 0 0))
+  )
   (wire (pts (xy 91.44 113.03) (xy 69.85 113.03))
     (stroke (width 0) (type default) (color 0 0 0 0))
@@
   (wire (pts (xy 91.44 52.07) (xy 69.85 52.07))
     (stroke (width 0) (type default) (color 0 0 0 0))
+  )
+  (text "pico pw sw en" (at 49.53 251.46 0)
+    (effects (font (size 1.27 1.27)) (justify left bottom))
   )
   (text "possible move these to microJSTs?" (at 135.89 137.16 0)
@@
     (effects (font (size 1.27 1.27) (thickness 0.254) bold) (justify left bottom))
   )
-  (text "enable openLST" (at 41.91 254 0)
+  (text "irridum OnOff (high pulls low)" (at 49.53 241.3 0)
     (effects (font (size 1.27 1.27)) (justify left bottom))
   )
@@
     (effects (font (size 1.27 1.27)) (justify left bottom))
   )
-  (text "regular GPIO" (at 41.91 232.41 0)
+  (text "regular GPIO" (at 22.86 228.6 0)
     (effects (font (size 1.27 1.27)) (justify left bottom))
   )
@@
   (text "More efficient RF regulator,\nour more active Tx for streaming data\nmakes low eff lin reg more costly"
     (at 233.68 248.92 0)
+    (effects (font (size 1.27 1.27)) (justify left bottom))
+  )
+  (text "startracker pw sw en" (at 49.53 246.38 0)
+    (effects (font (size 1.27 1.27)) (justify left bottom))
+  )
+  (text "startracker RST" (at 49.53 248.92 0)
     (effects (font (size 1.27 1.27)) (justify left bottom))
   )
@@
     (effects (font (size 1.27 1.27)) (justify left bottom))
   )
-  (text "GPIO can also be ADC inputs" (at 41.91 215.9 0)
+  (text "GPIO can also be ADC inputs" (at 22.86 213.36 0)
     (effects (font (size 1.27 1.27)) (justify left bottom))
   )
@@
   (text "installing this \njumper will allow \ndata but disable \nusb source"
     (at 240.03 144.78 0)
+    (effects (font (size 1.27 1.27)) (justify left bottom))
+  )
+  (text "payload RST" (at 49.53 236.22 0)
     (effects (font (size 1.27 1.27)) (justify left bottom))
   )
@@
     (effects (font (size 1.27 1.27)) (justify left bottom))
   )
-  (text "currently unused, going to go somehwere eventually?"
-    (at 22.86 212.09 0)
-    (effects (font (size 1.27 1.27) (thickness 0.254) bold) (justify left bottom))
-  )
   (text "green led turns on when 5Vusb is high" (at 189.23 26.67 0)
     (effects (font (size 1.27 1.27)) (justify left bottom))
@@
     (effects (font (size 2.54 2.54) (thickness 0.508) bold) (justify left bottom))
   )
-  (text "enable irridium" (at 41.91 251.46 0)
+  (text "irridum pw sw en" (at 49.53 238.76 0)
     (effects (font (size 1.27 1.27)) (justify left bottom))
   )
   (text "Vbatt_RET" (at 115.57 113.03 0)
+    (effects (font (size 1.27 1.27)) (justify left bottom))
+  )
+  (text "payload pw sw en" (at 49.53 243.84 0)
     (effects (font (size 1.27 1.27)) (justify left bottom))
   )
@@
     (effects (font (size 1.27 1.27)) (justify left bottom))
   )
+  (text "payload SERVO_PWR_CTRL" (at 49.53 233.68 0)
+    (effects (font (size 1.27 1.27)) (justify left bottom))
+  )
   (text "Payload regulator (also magnetotorqer and wheel(s))"
     (at 102.87 262.89 0)
@@
     )
   )
-  (global_label "BP_LED_LATCH" (shape bidirectional) (at 44.45 257.81 0) (fields_autoplaced)
-    (effects (font (size 1.27 1.27)) (justify left))
-    (property "Intersheet References" "${INTERSHEET_REFS}" (id 0) (at 0 0 0)
-      (effects (font (size 1.27 1.27)) hide)
-    )
-  )
   (global_label "VBUS_INHIBIT" (shape bidirectional) (at 252.73 55.88 180) (fields_autoplaced)
     (effects (font (size 1.27 1.27)) (justify right))
@@
     (property "Intersheet References" "${INTERSHEET_REFS}" (id 0) (at 0 0 0)
       (effects (font (size 1.27 1.27)) hide)
+    )
+  )
+  (global_label "NeoPixel_Out" (shape input) (at 44.45 257.81 0) (fields_autoplaced)
+    (effects (font (size 1.27 1.27)) (justify left))
+    (property "Intersheet References" "${INTERSHEET_REFS}" (id 0) (at 59.1718 257.8894 0)
+      (effects (font (size 1.27 1.27)) (justify left) hide)
     )
   )
@@
     (pin "2")
   )
-  (symbol (lib_id "mainboard-rescue:Q_NPN_BCE-Device-mainboard-rescue") (at 275.59 168.91 0) (unit 1)
+  (symbol (lib_id "mainboard-rescue:Q_NPN_BEC-Device-mainboard-rescue") (at 275.59 168.91 0) (unit 1)
     (in_bom yes) (on_board yes)
     (property "Reference" "Q205" (id 0) (at 280.4414 167.7416 0)

Commit message: friday updates
Parts:
- removed J201: TSM-102-01-L-SV-P-TR, Connector_PinSocket_2.54mm:PinSocket_1x02_P2.54mm_Vertical_SMD_Pin1Right, symbol Connector_Generic:Conn_01x02
- added R9: 100, Resistor_SMD:R_0603_1608Metric, symbol Device:R_US
- R12, R16: renamed from R?; footprint (none) -> Resistor_SMD:R_0603_1608Metric
- gave numbers to parts that had none: 5
Connections:
- net VBATT: no longer Q207.5 (D), Q207.6 (D), Q207.7 (D), Q207.8 (D)
- net ~{USB_EN}: now also R9.1
- net PC00 renamed AIN10
- net PC01 renamed AIN11
- net PC02 renamed AIN4
- net SELF_TEST renamed ~{SELF_TEST}
- new net Blank-Card-Default/~{USB_EN}: R9.2
- new net VCHRG: Q207.5 (D), Q207.6 (D), Q207.7 (D), Q207.8 (D)
Other:
- note added: "(no RBF) & (sep1 open) & (sep2 open) & (sep3 open) = main bus powered"
- note added: "5Vusb + RBF = usb battery charge bus unpowered"
- note added: "5Vusb + no RBF = usb battery charge and powers bus"
- note added: "RBF installed = pulled to GNDREF"
- note added: "SEP1 low = gate high = on"
- note added: "high side bus sw"
- note added: "high side chg sw"
- note added: "low side bus sw"
- note added: "quadruple triple double check these"
- note added: "rbf low = gate low = on"
- note added: "self test routine button, pulled up at MCU"
- note added: "sep2 low = gate low = on"
- note added: "sep3 low = gate low = on"
- note added: "wouldnt tie-ing RBD to R219 do the trick?"
- note removed: "(RBF open) & (sep1 open) & (sep2 open) & (sep3 open) = main bus powered"
- note removed: "5Vusb + RBF installed = usb battery charge bus unpowered"
- note removed: "5Vusb + RBF not installed = usb battery charge and powers bus"
- note removed: "installing this jumper will allow data but disable usb source"

Commit message: text changes
Other:
- note added: "rbf HiZ = pnp off = gate low = on"
- note removed: "rbf low = gate low = on"
Changed lines of the file:
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@@
     (stroke (width 0) (type default) (color 0 0 0 0))
   )
-  (text "rbf low = gate low = on" (at 383.54 96.52 0)
+  (text "rbf HiZ = pnp off = gate low = on" (at 382.27 97.79 0)
     (effects (font (size 1.27 1.27)) (justify left bottom))
   )

Commit message: fm sch changes
Parts:
- removed Q14: MMBT3906-7-F, Package_TO_SOT_SMD:SOT-23, symbol mainboard-rescue:Q_PNP_BEC-Device-mainboard-rescue
- removed Q205: MMBT4401-7-F, Package_TO_SOT_SMD:SOT-23, symbol mainboard-rescue:Q_NPN_BEC-Device-mainboard-rescue
- removed Q206: IRF7458, Package_SO:SOIC-8_3.9x4.9mm_P1.27mm, symbol mainboard_SLI:IRF7458
- removed R12: 100k, Resistor_SMD:R_0603_1608Metric, symbol Device:R_US
- removed R16: 2.2Meg, Resistor_SMD:R_0603_1608Metric, symbol Device:R_US
- removed R213: 100k, Resistor_SMD:R_0603_1608Metric, symbol mainboard-rescue:R_US-Device-mainboard-rescue
- removed R214, R248: 2.2Meg, Resistor_SMD:R_0603_1608Metric, symbol mainboard-rescue:R_US-Device-mainboard-rescue
- added Q51: MMBT4401-7-F, Package_TO_SOT_SMD:SOT-23, symbol mainboard-rescue:Q_NPN_BEC-Device-mainboard-rescue
- added Q52, Q53, Q54: MMBT3906-7-F, Package_TO_SOT_SMD:SOT-23, symbol mainboard-rescue:Q_PNP_BEC-Device-mainboard-rescue
- added R102, R106: 100k, Resistor_SMD:R_0603_1608Metric, symbol Device:R_US
- added R103: 1Meg, Resistor_SMD:R_0603_1608Metric, symbol Device:R_US
- added R105, R57: 10k, Resistor_SMD:R_0603_1608Metric, symbol Device:R_US
- added R111, R112, R113, R58: 100, Resistor_SMD:R_0603_1608Metric, symbol Device:R_US
- R10: symbol mainboard-rescue:R_US-Device-mainboard-rescue -> Device:R_US
- R11, R216, R219, R220, R221: value 2.2Meg -> 1Meg; symbol mainboard-rescue:R_US-Device-mainboard-rescue -> Device:R_US
- R218: value 100k -> 10k; symbol mainboard-rescue:R_US-Device-mainboard-rescue -> Device:R_US
Connections:
- net 5V_USB: now also Q51.3 (C), R57.2
- net GNDREF: now also Q53.3 (C), R103.2
- net RBF: now also R102.2, R105.2; no longer R218.2
- net SEP2: now also R111.1; no longer Q211.4 (G)
- net SEP3: now also R112.1; no longer Q212.4 (G)
- net SEP4: now also R218.2, R106.2
- net VBUS_INHIBIT: now also Q52.2 (E), Q54.2 (E)
- net at Q9.3 (C), R11.1: now also Q51.2 (E), R58.1; no longer Q208.4 (G)
- net at Q207.4 (G), R216.2: now also Q53.2 (E)
- net at Q220.4 (G): now also R113.2
- net +X_SOLAR_TLE renamed SLR_TLE_3
- net +Y_SOLAR_TLE renamed SLR_TLE_1
- net -X_SOLAR_TLE renamed SLR_TLE_2
- net -Z_SOLAR_TLE renamed SLR_TLE_4
- new net: Q208.4 (G), R58.2
- new net: Q211.4 (G), R111.2
- new net: Q212.4 (G), R112.2
- new net: Q52.1 (B), R102.1
- new net: Q52.3 (C), Q54.3 (C), R103.1, R113.1
- new net: Q54.1 (B), R106.1
- new net: Q53.1 (B), R105.1
- new net: Q51.1 (B), R57.1
Other:
- sheet Payload_Regulator ports: added NTC; removed none
- sheet RF_Regulator ports: added NTC; removed none
- note added: "1. no RBF + sep4 hiZ = no charge, bus not powered by vbus usb (flight) 2. 5Vusb + no RBF + sep4 low = no charge, bus powered by 5Vusb(debug WITHOUT battery) 3. 5Vusb + RBF + sep4 hiZ = charge, bus unpowered (ground charge) 4. 5Vusb + RBF + sep4 low = charge, bus powered by ONLY 5Vusb (debug) do NOT have a battery connected during #2"
- note added: "Payload regulator"
- note added: "RBF is N/O to gnd (install pulls RBF to gndref)"
- note added: "RF regulator"
- note added: "SEP4 is not used on the sat, but used to for debug mode"
- note added: "rbf and sep4 HiZ = pnp off = on"
- note added: "solar panel TLE inputs lm355A temp sensors on panels"
- note removed: "5Vusb + RBF = usb battery charge bus unpowered"
- note removed: "5Vusb + no RBF = usb battery charge and powers bus"
- note removed: "GNDREF is battery return"
- note removed: "More efficient RF regulator, our more active Tx for streaming data makes low eff lin reg more costly"
- note removed: "Payload regulator (also magnetotorqer and wheel(s))"
- note removed: "RBF installed = pulled to GNDREF"
- note removed: "RBF is N/O to gnd (install pulls RBF low)"
- note removed: "RF regulator replacement (more efficient)"
- note removed: "SEP1 low = gate high = on"
- note removed: "fix this ckt"
- note removed: "low side bus sw"
- note removed: "quadruple triple double check these"
- note removed: "rbf HiZ = pnp off = gate low = on"
- note removed: "wouldnt tie-ing RBD to R219 do the trick?"
- moved on the sheet: Q10, Q207, Q208, Q211, Q212, Q213, Q220, Q9, R10, R11, R216, R218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

Commit message: fm layout work
Changed lines of the file:
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@@
+    (pin "1")
+  )
+  (symbol (lib_id "mainboard-rescue:GNDREF-power-mainboard-rescue") (at 111.76 69.85 0) (unit 1)
+    (in_bom yes) (on_board yes)
+    (property "Reference" "#PWR0106" (id 0) (at 111.76 76.2 0)
+      (effects (font (size 1.27 1.27)) hide)
+    )
+    (property "Value" "GNDREF" (id 1) (at 111.887 74.2442 0))
+    (property "Footprint" "" (id 2) (at 111.76 69.85 0)
+      (effects (font (size 1.27 1.27)) hide)
+    )
+    (property "Datasheet" "" (id 3) (at 111.76 69.85 0)
+      (effects (font (size 1.27 1.27)) hide)
+    )
     (pin "1")
   )

Commit message: more fm layout
Parts:
- removed R9: 100, Resistor_SMD:R_0603_1608Metric, symbol Device:R_US
- added R134, R135: 100, Resistor_SMD:R_0603_1608Metric, symbol Device:R_US
Connections:
- net at Q10.2 (E), R219.2: now also R134.1; no longer Q213.4 (G)
- net at Q53.2 (E), R216.2: now also R135.1; no longer Q207.4 (G)
- new net: Q213.4 (G), R134.2
- new net: Q207.4 (G), R135.2
Changed lines of the file:
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@@
-    (stroke (width 0) (type default) (color 0 0 0 0))
-  )
-  (wire (pts (xy 285.75 154.94) (xy 273.05 154.94))
     (stroke (width 0) (type default) (color 0 0 0 0))
   )
@@
     (stroke (width 0) (type default) (color 0 0 0 0))
   )
-  (wire (pts (xy 367.03 153.67) (xy 355.6 153.67))
-    (stroke (width 0) (type default) (color 0 0 0 0))
-  )
   (polyline (pts (xy 148.59 146.05) (xy 148.59 154.94))
     (stroke (width 0) (type default) (color 0 0 0 0))
@@
     (stroke (width 0) (type default) (color 0 0 0 0))
   )
-  (wire (pts (xy 123.19 38.1) (xy 144.78 38.1))
+  (wire (pts (xy 119.38 38.1) (xy 144.78 38.1))
     (stroke (width 0) (type default) (color 0 0 0 0))
   )
@@
     (stroke (width 0) (type default) (color 0 0 0 0))
   )
+  (wire (pts (xy 359.41 153.67) (xy 355.6 153.67))
+    (stroke (width 0) (type default) (color 0 0 0 0))
+  )
   (polyline (pts (xy 166.37 234.95) (xy 166.37 252.73))
     (stroke (width 0) (type default) (color 0 0 0 0))
@@
     (stroke (width 0) (type default) (color 0 0 0 0))
   )
-  (wire (pts (xy 111.76 38.1) (xy 115.57 38.1))
-    (stroke (width 0) (type default) (color 0 0 0 0))
-  )
   (wire (pts (xy 119.38 127) (xy 119.38 121.92))
     (stroke (width 0) (type default) (color 0 0 0 0))
@@
   )
   (wire (pts (xy 165.1 125.73) (xy 172.72 125.73))
+    (stroke (width 0) (type default) (color 0 0 0 0))
+  )
+  (wire (pts (xy 278.13 154.94) (xy 273.05 154.94))
     (stroke (width 0) (type default) (color 0 0 0 0))
   )
@@
     )
   )
-  (global_label "~{USB_EN}" (shape input) (at 111.76 38.1 180) (fields_autoplaced)
+  (global_label "~{USB_EN}" (shape input) (at 119.38 38.1 180) (fields_autoplaced)
     (effects (font (size 1.27 1.27)) (justify right))
-    (property "Intersheet References" "${INTERSHEET_REFS}" (id 0) (at 102.1787 38.0206 0)
+    (property "Intersheet References" "${INTERSHEET_REFS}" (id 0) (at 109.7987 38.0206 0)
       (effects (font (size 1.27 1.27)) (justify right) hide)
     )
@@
     (pin "3")
   )
+  (symbol (lib_id "Device:R_US") (at 363.22 153.67 90) (unit 1)
+    (in_bom yes) (on_board yes) (fields_autoplaced)
+    (property "Reference" "R135" (id 0) (at 363.22 147.32 90))
+    (property "Value" "100" (id 1) (at 363.22 149.86 90))
+    (property "Footprint" "Resistor_SMD:R_0603_1608Metric" (id 2) (at 363.474 152.654 90)
+      (effects (font (size 1.27 1.27)) hide)
+    )
+    (property "Datasheet" "~" (id 3) (at 363.22 153.67 0)
+      (effects (font (size 1.27 1.27)) hide)
+    )
+    (pin "1")
+    (pin "2")
+  )
   (symbol (lib_id "Device:R_US") (at 341.63 161.29 270) (unit 1)
     (in_bom yes) (on_board yes)
@@
     (pin "2")
   )
-  (symbol (lib_id "Device:R_US") (at 119.38 38.1 90) (unit 1)
+  (symbol (lib_id "Device:R_US") (at 281.94 154.94 90) (unit 1)
     (in_bom yes) (on_board yes) (fields_autoplaced)
-    (property "Reference" "R9" (id 0) (at 119.38 31.75 90))
-    (property "Value" "100" (id 1) (at 119.38 34.29 90))
-    (property "Footprint" "Resistor_SMD:R_0603_1608Metric" (id 2) (at 119.634 37.084 90)
-      (effects (font (size 1.27 1.27)) hide)
-    )
-    (property "Datasheet" "~" (id 3) (at 119.38 38.1 0)
-      (effects (font (size 1.27 1.27)) hide)
-    )
+    (property "Reference" "R134" (id 0) (at 281.94 148.59 90))
+    (property "Value" "100" (id 1) (at 281.94 151.13 90))
+    (property "Footprint" "Resistor_SMD:R_0603_1608Metric" (id 2) (at 282.194 153.924 90)
+      (effects (font (size 1.27 1.27)) hide)
+    )
+    (property "Datasheet" "~" (id 3) (at 281.94 154.94 0)
+      (effects (font (size 1.27 1.27)) hide)
+    )
