File: hardware/foras-promineo-revB-fm/analog_mux.kicad_sch (KiCad schematic)
At the start: 24 parts, among them U6 74HC4067PW,118, U7 OPA340MDBVTEP

Commit message: preparing for battery testing
Parts:
- R58: value 100k -> 110k
Changed lines of the file:
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@@
       (effects (font (size 1.27 1.27)) (justify left))
     )
-    (property "Value" "100k" (id 1) (at 74.93 66.0399 0)
+    (property "Value" "110k" (id 1) (at 74.93 66.0399 0)
       (effects (font (size 1.27 1.27)) (justify left))
     )

Commit message: fm sch changes
Parts:
- removed R39, R40: 100k, Resistor_SMD:R_0603_1608Metric, symbol Device:R_US
- removed R57: 330k, Resistor_SMD:R_0603_1608Metric, symbol Device:R_US
- removed R58: 110k, Resistor_SMD:R_0603_1608Metric, symbol Device:R_US
- added J52: samtec x, symbol Connector_Generic:Conn_02x04_Odd_Even
- added R117, R118, R123, R124, R129, R130, R131, R132: 100k, Resistor_SMD:R_0603_1608Metric, symbol Device:R_US
- added R119, R121, R125, R127: 10k, Resistor_SMD:R_0603_1608Metric, symbol Device:R_US
- added R120, R122, R126, R128: 1k, Resistor_SMD:R_0603_1608Metric, symbol Device:R_US
- C22, C9: symbol mainboard-rescue:C-Device-mainboard-rescue -> Device:C
Connections:
- net VBAT_adc is gone; now on net VSOLAR_adc: U6.6 (I3)
- net 3.3V: now also R119.1, R121.1, R125.1, R127.1
- net GND: now also J52.2 (Pin_2), J52.4 (Pin_4), J52.6 (Pin_6), J52.8 (Pin_8), R118.2, R124.2, R130.2, R132.2
- net VCC_PAYLOAD: now also R120.1, R122.1, R126.1, R128.1
- net VSOLAR_adc: no longer U6.5 (I4)
- net slr_temp_4: now reaches U6.16 (I15)
- net slr_temp_4: now also R131.2, R132.1
- net slr_temp_3: now reaches U6.17 (I14)
- net slr_temp_3: now also R129.2, R130.1
- net slr_temp_2: now reaches U6.18 (I13)
- net slr_temp_2: now also R123.2, R124.1
- net slr_temp_1: now reaches U6.19 (I12)
- net slr_temp_1: now also R117.2, R118.1
- net VRF_NTC: now reaches U6.2 (I7)
- net NTC4: now reaches U6.20 (I11)
- net NTC4: now also J52.7 (Pin_7), R119.2
- net NTC3: now reaches U6.21 (I10)
- net NTC3: now also J52.5 (Pin_5), R121.2
- net NTC2: now reaches U6.22 (I9)
- net NTC2: now also J52.3 (Pin_3), R125.2
- net NTC1: now reaches U6.23 (I8)
- net NTC1: now also J52.1 (Pin_1), R127.2
- net VPYLD_NTC: now reaches U6.3 (I6)
- net SLR_CHRG_NTC: now reaches U6.4 (I5)
- new net BATT_NTC: U6.5 (I4)
- new net SLR_TLE_1: R117.1, R120.2, R123.1, R129.1, R131.1
- new net SLR_TLE_2: R122.2
- new net SLR_TLE_3: R126.2
- new net SLR_TLE_4: R128.2
Other:
- note added: "lm355a is rated to 100degC arbitrarily selecting max temp sensed as 400K ~ 125C"
- note added: "really should have an op amp here but board space is already constrained"
- note removed: "add NTCs around each regulator?"
- moved on the sheet: R59, R65

Commit message: fm layout work
Parts:
- J52: value samtec x -> T1M-08-F-SV-L; footprint (none) -> mainboard-SLI:SAMTEC_T1M-08-F-SV-L
Changed lines of the file:
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@@
     (in_bom yes) (on_board yes) (fields_autoplaced)
     (property "Reference" "J52" (id 0) (at 80.01 93.98 0))
-    (property "Value" "samtec x" (id 1) (at 80.01 96.52 0))
-    (property "Footprint" "" (id 2) (at 78.74 105.41 0)
+    (property "Value" "T1M-08-F-SV-L" (id 1) (at 80.01 96.52 0))
+    (property "Footprint" "mainboard-SLI:SAMTEC_T1M-08-F-SV-L" (id 2) (at 78.74 105.41 0)
       (effects (font (size 1.27 1.27)) hide)
     )
-    (property "Datasheet" "~" (id 3) (at 78.74 105.41 0)
+    (property "Datasheet" "T1M-08-F-SV-L" (id 3) (at 78.74 105.41 0)
       (effects (font (size 1.27 1.27)) hide)
     )

Commit message: more fm layout
Parts:
- removed R20, R31: 100k, Resistor_SMD:R_0603_1608Metric, symbol Device:R_US
Connections:
- net SLR_TLE_1: no longer R123.1, R129.1, R131.1
- net SLR_TLE_2: now also R123.1
- net SLR_TLE_3: now also R129.1
- net SLR_TLE_4: now also R131.1
- net 3.3V_adc: no longer names the net of U6.9 (I0)
- no-connect marks 0 -> 1
Changed lines of the file:
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@@
   (junction (at 203.2 45.72) (diameter 0) (color 0 0 0 0)
   )
-  (junction (at 20.32 59.69) (diameter 0) (color 0 0 0 0)
-  )
   (junction (at 54.61 179.07) (diameter 0) (color 0 0 0 0)
   )
@@
   (junction (at 41.91 110.49) (diameter 0) (color 0 0 0 0)
   )
+  (no_connect (at 172.72 72.39))
   (wire (pts (xy 172.72 102.87) (xy 176.53 102.87))
     (stroke (width 0) (type default) (color 0 0 0 0))
@@
     (stroke (width 0) (type default) (color 0 0 0 0))
   )
-  (wire (pts (xy 20.32 49.53) (xy 20.32 50.8))
-    (stroke (width 0) (type default) (color 0 0 0 0))
-  )
   (wire (pts (xy 41.91 97.79) (xy 41.91 110.49))
     (stroke (width 0) (type default) (color 0 0 0 0))
@@
     (stroke (width 0) (type default) (color 0 0 0 0))
   )
-  (wire (pts (xy 20.32 58.42) (xy 20.32 59.69))
-    (stroke (width 0) (type default) (color 0 0 0 0))
-  )
   (wire (pts (xy 127 105.41) (xy 132.08 105.41))
     (stroke (width 0) (type default) (color 0 0 0 0))
@@
     (stroke (width 0) (type default) (color 0 0 0 0))
   )
-  (wire (pts (xy 20.32 59.69) (xy 20.32 60.96))
-    (stroke (width 0) (type default) (color 0 0 0 0))
-  )
   (wire (pts (xy 86.36 105.41) (xy 86.36 107.95))
     (stroke (width 0) (type default) (color 0 0 0 0))
@@
     (stroke (width 0) (type default) (color 0 0 0 0))
   )
-  (wire (pts (xy 20.32 59.69) (xy 22.86 59.69))
-    (stroke (width 0) (type default) (color 0 0 0 0))
-  )
   (wire (pts (xy 39.37 130.81) (xy 43.18 130.81))
     (stroke (width 0) (type default) (color 0 0 0 0))
@@
   )
   (wire (pts (xy 107.95 168.91) (xy 109.22 168.91))
-    (stroke (width 0) (type default) (color 0 0 0 0))
-  )
-  (wire (pts (xy 172.72 72.39) (xy 181.61 72.39))
     (stroke (width 0) (type default) (color 0 0 0 0))
   )
@@
     (effects (font (size 1.27 1.27)) (justify left bottom))
   )
-  (label "3.3V_adc" (at 181.61 72.39 0)
-    (effects (font (size 1.27 1.27)) (justify left bottom))
-  )
   (label "NTC1" (at 63.5 102.87 180)
     (effects (font (size 1.27 1.27)) (justify right bottom))
@@
   (label "NTC3" (at 48.26 107.95 180)
     (effects (font (size 1.27 1.27)) (justify right bottom))
-  )
-  (label "3.3V_adc" (at 22.86 59.69 0)
-    (effects (font (size 1.27 1.27)) (justify left bottom))
   )
   (label "NTC4" (at 176.53 100.33 0)
@@
     )
   )
-  (global_label "SLR_TLE_1" (shape input) (at 107.95 168.91 180) (fields_autoplaced)
+  (global_label "SLR_TLE_4" (shape input) (at 107.95 168.91 180) (fields_autoplaced)
     (effects (font (size 1.27 1.27)) (justify right))
     (property "Intersheet References" "${INTERSHEET_REFS}" (id 0) (at 95.8287 168.8306 0)
@@
     )
   )
-  (global_label "SLR_TLE_1" (shape input) (at 78.74 168.91 180) (fields_autoplaced)
+  (global_label "SLR_TLE_3" (shape input) (at 78.74 168.91 180) (fields_autoplaced)
     (effects (font (size 1.27 1.27)) (justify right))
     (property "Intersheet References" "${INTERSHEET_REFS}" (id 0) (at 66.6187 168.8306 0)
@@
     )
   )
-  (global_label "SLR_TLE_1" (shape input) (at 53.34 168.91 180) (fields_autoplaced)
+  (global_label "SLR_TLE_2" (shape input) (at 53.34 168.91 180) (fields_autoplaced)
     (effects (font (size 1.27 1.27)) (justify right))
     (property "Intersheet References" "${INTERSHEET_REFS}" (id 0) (at 41.2187 168.8306 0)
@@
     (pin "1")
   )
-  (symbol (lib_id "Device:R_US") (at 20.32 64.77 0) (unit 1)
-    (in_bom yes) (on_board yes) (fields_autoplaced)
-    (property "Reference" "R31" (id 0) (at 22.86 63.4999 0)
-      (effects (font (size 1.27 1.27)) (justify left))
-    )
-    (property "Value" "100k" (id 1) (at 22.86 66.0399 0)
-      (effects (font (size 1.27 1.27)) (justify left))
-    )
-    (property "Footprint" "Resistor_SMD:R_0603_1608Metric" (id 2) (at 21.336 65.024 90)
-      (effects (font (size 1.27 1.27)) hide)
-    )
-    (property "Datasheet" "~" (id 3) (at 20.32 64.77 0)
-      (effects (font (size 1.27 1.27)) hide)
-    )
-    (pin "1")
-    (pin "2")
-  )
   (symbol (lib_id "mainboard:GND") (at 143.51 66.04 0) (unit 1)
     (in_bom yes) (on_board yes)
@@
     (pin "1")
     (pin "2")
-  )
-  (symbol (lib_id "mainboard:3.3V") (at 20.32 49.53 0) (unit 1)
-    (in_bom yes) (on_board yes)
-    (property "Reference" "#SUPPLY0126" (id 0) (at 20.32 49.53 0)
-      (effects (font (size 1.27 1.27)) hide)
-    )
-    (property "Value" "3.3V" (id 1) (at 17.78 45.72 0)
-      (effects (font (size 1.4986 1.4986)) (justify left bottom))
-    )
-    (property "Footprint" "" (id 2) (at 20.32 49.53 0)
-      (effects (font (size 1.27 1.27)) hide)
-    )
-    (property "Datasheet" "" (id 3) (at 20.32 49.53 0)
-      (effects (font (size 1.27 1.27)) hide)
-    )
-    (pin "1")
   )
   (symbol (lib_id "mainboard:3.3V") (at 143.51 55.88 0) (unit 1)
@@
     (pin "2")
   )
-  (symbol (lib_id "Device:R_US") (at 20.32 54.61 0) (unit 1)
-    (in_bom yes) (on_board yes) (fields_autoplaced)
-    (property "Reference" "R20" (id 0) (at 22.86 53.3399 0)
-      (effects (font (size 1.27 1.27)) (justify left))
-    )
-    (property "Value" "100k" (id 1) (at 22.86 55.8799 0)
-      (effects (font (size 1.27 1.27)) (justify left))
-    )
-    (property "Footprint" "Resistor_SMD:R_0603_1608Metric" (id 2) (at 21.336 54.864 90)
-      (effects (font (size 1.27 1.27)) hide)
-    )
-    (property "Datasheet" "~" (id 3) (at 20.32 54.61 0)
-      (effects (font (size 1.27 1.27)) hide)
-    )
-    (pin "1")
-    (pin "2")
-  )
   (symbol (lib_id "Device:C") (at 203.2 49.53 0) (unit 1)
     (in_bom yes) (on_board yes)
@@
     (pin "2")
   )
-  (symbol (lib_id "mainboard:GND") (at 20.32 71.12 0) (unit 1)
-    (in_bom yes) (on_board yes)
-    (property "Reference" "#GND0127" (id 0) (at 20.32 71.12 0)
-      (effects (font (size 1.27 1.27)) hide)
-    )
-    (property "Value" "GND" (id 1) (at 17.78 73.66 0)
-      (effects (font (size 1.4986 1.4986)) (justify left bottom))
-    )
-    (property "Footprint" "" (id 2) (at 20.32 71.12 0)
-      (effects (font (size 1.27 1.27)) hide)
-    )
-    (property "Datasheet" "" (id 3) (at 20.32 71.12 0)
-      (effects (font (size 1.27 1.27)) hide)
-    )
-    (pin "1")
-  )
   (symbol (lib_id "Device:R_US") (at 109.22 173.99 0) (unit 1)
