File: hardware/foras-promineo-revB-fm/mainboard.kicad_sch (KiCad schematic)
At the start: 0 parts

Commit message: more tweaking
Changed lines of the file:
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@@
     (stroke (width 0) (type default) (color 0 0 0 0))
   )
-  (text "SLI ADDED" (at 148.59 40.64 0)
+  (text "SLI ADDED" (at 165.1 40.64 0)
     (effects (font (size 1.27 1.27)) (justify left bottom))
   )
@@
     )
   )
-  (sheet (at 144.78 20.32) (size 58.42 21.59) (fields_autoplaced)
+  (sheet (at 161.29 20.32) (size 58.42 21.59) (fields_autoplaced)
     (stroke (width 0) (type solid) (color 0 0 0 0))
     (fill (color 0 0 0 0.0000))
-    (property "Sheet name" "Solar Charge Regulator" (id 0) (at 144.78 18.9734 0)
+    (property "Sheet name" "Solar Charge Regulator" (id 0) (at 161.29 18.9734 0)
       (effects (font (size 2.54 2.54)) (justify left bottom))
     )
-    (property "Sheet file" "Solar Charge Regulator.kicad_sch" (id 1) (at 144.78 43.0026 0)
+    (property "Sheet file" "Solar Charge Regulator.kicad_sch" (id 1) (at 161.29 43.0026 0)
       (effects (font (size 2.54 2.54)) (justify left top))
     )

Commit message: friday updates
Other:
- added sheet analog_mux (analog_mux.kicad_sch)

Commit message: fm sch changes
Other:
- sheet analog_mux renamed adc_mux
