File: hardware/foras-promineo-revB-em/5V_regulator.kicad_sch (KiCad schematic)
At the start: 17 parts, among them Q222 MMBT3906-7-F, U210 TPS63070

Commit message: em design complete
todo: update BOM
Parts:
- L202: footprint Inductor_SMD:L_Bourns_SRN8040TA -> mainboard-SLI:L_Bourns_SRN8040TA
Changed lines of the file:
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@@
       (effects (font (size 1.27 1.27)) (justify left))
     )
-    (property "Footprint" "Inductor_SMD:L_Bourns_SRN8040TA" (id 2) (at 170.18 52.07 0)
+    (property "Footprint" "mainboard-SLI:L_Bourns_SRN8040TA" (id 2) (at 170.18 52.07 0)
       (effects (font (size 1.27 1.27)) hide)
     )
