File: hardware/foras-promineo-revB-em/Avionics.kicad_sch (KiCad schematic)
At the start: 33 parts, among them SW1 KMR231NG LFS, U1 MAX706RESA, U2 ATSAMD51N20A-AUT, Y1 32.768kHz

Commit message: em design complete
todo: update BOM
Other:
- note removed: "rts/cts pins can also be serial ports, future flexability"
Changed lines of the file:
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@@
     (stroke (width 0) (type default) (color 0 0 0 0))
   )
-  (polyline (pts (xy 180.34 73.66) (xy 180.34 93.98))
+  (polyline (pts (xy 180.34 73.66) (xy 180.34 90.17))
     (stroke (width 0) (type default) (color 0 0 0 0))
   )
@@
   (text "SDA2" (at 73.66 87.63 0)
     (effects (font (size 0.889 0.889)) (justify left bottom))
-  )
-  (text "rts/cts pins can also be serial ports, future flexability "
-    (at 157.48 97.79 0)
-    (effects (font (size 1.27 1.27)) (justify left bottom))
   )
   (text "DNI SW1\nSW200 is the rst switch now" (at 17.78 17.78 0)
@@
   )
   (global_label "ENAB_BURN1" (shape bidirectional) (at 146.05 107.95 0) (fields_autoplaced)
-    (effects (font (size 0.9906 0.9906)) (justify left))
-    (property "Intersheet References" "${INTERSHEET_REFS}" (id 0) (at 0 0 0)
-      (effects (font (size 1.27 1.27)) hide)
+    (effects (font (size 1.27 1.27)) (justify left))
+    (property "Intersheet References" "${INTERSHEET_REFS}" (id 0) (at 160.5904 107.8706 0)
+      (effects (font (size 1.27 1.27)) (justify left) hide)
     )
   )
@@
   )
   (global_label "BURN_RELAY_A" (shape bidirectional) (at 146.05 105.41 0) (fields_autoplaced)
-    (effects (font (size 0.9906 0.9906)) (justify left))
-    (property "Intersheet References" "${INTERSHEET_REFS}" (id 0) (at 0 0 0)
-      (effects (font (size 1.27 1.27)) hide)
-    )
-  )
+    (effects (font (size 1.27 1.27)) (justify left))
+    (property "Intersheet References" "${INTERSHEET_REFS}" (id 0) (at 162.2232 105.3306 0)
+      (effects (font (size 1.27 1.27)) (justify left) hide)
+    )
+  )
