File: hardware/foras-promineo-revB-em/Power.kicad_sch (KiCad schematic)
At the start: 43 parts, among them Q1 DMN100-7-F, Q2 MMDT5551-7-F, Q22 IRF7404TRPBF, Q3 MMDT5551-7-F, U17 BQ25883RGER, U4 ADM1176-1ARMZ-R7, U5 TPS54226PWPRPWP14_2P31X2P46-L

Commit message: em design complete
todo: update BOM
Parts:
- added R167: 100k, Resistor_SMD:R_0603_1608Metric, symbol Device:R_US
Connections:
- net GNDREF: now also R167.2
- net at U17.3 (~{CE}): now also R167.1
- no-connect marks 5 -> 4
Changed lines of the file:
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@@
   (no_connect (at 223.52 138.43))
   (no_connect (at 226.06 138.43))
-  (no_connect (at 210.82 115.57))
   (wire (pts (xy 54.61 166.37) (xy 62.23 166.37))
     (stroke (width 0) (type default) (color 0 0 0 0))
@@
   )
   (wire (pts (xy 127 102.87) (xy 127 97.79))
+    (stroke (width 0) (type default) (color 0 0 0 0))
+  )
+  (wire (pts (xy 190.5 115.57) (xy 210.82 115.57))
     (stroke (width 0) (type default) (color 0 0 0 0))
   )
@@
     (pin "9")
   )
+  (symbol (lib_id "mainboard-rescue:GNDREF-power-mainboard-rescue") (at 190.5 123.19 0) (unit 1)
+    (in_bom yes) (on_board yes)
+    (property "Reference" "#PWR0106" (id 0) (at 190.5 129.54 0)
+      (effects (font (size 1.27 1.27)) hide)
+    )
+    (property "Value" "GNDREF" (id 1) (at 190.627 127.5842 0))
+    (property "Footprint" "" (id 2) (at 190.5 123.19 0)
+      (effects (font (size 1.27 1.27)) hide)
+    )
+    (property "Datasheet" "" (id 3) (at 190.5 123.19 0)
+      (effects (font (size 1.27 1.27)) hide)
+    )
+    (pin "1")
+  )
+  (symbol (lib_id "Device:R_US") (at 190.5 119.38 0) (mirror y) (unit 1)
+    (in_bom yes) (on_board yes)
+    (property "Reference" "R167" (id 0) (at 188.7982 118.2116 0)
+      (effects (font (size 1.27 1.27)) (justify left))
+    )
+    (property "Value" "100k" (id 1) (at 188.7982 120.523 0)
+      (effects (font (size 1.27 1.27)) (justify left))
+    )
+    (property "Footprint" "Resistor_SMD:R_0603_1608Metric" (id 2) (at 189.484 119.634 90)
+      (effects (font (size 1.27 1.27)) hide)
+    )
+    (property "Datasheet" "" (id 3) (at 190.5 119.38 0)
+      (effects (font (size 1.27 1.27)) hide)
+    )
+    (property "Description" "" (id 4) (at 188.7982 115.6716 0)
+      (effects (font (size 1.27 1.27)) hide)
+    )
+    (pin "1")
+    (pin "2")
+  )
 )
