File: hardware/foras-promineo-revB-em/Solar Charge Regulator.kicad_sch (KiCad schematic)
At the start: 27 parts, among them U211 ‎LT3652HVEMSE#TRPBF‎, U3 ADM1176-1ARMZ-R7

Commit message: em2 stuff
Other:
- note added: "RIN1/RIN2 = (VIN(MIN)/2.7) – 1 these set the MPP for the cells"
- note removed: "RIN1/RIN2 = (VIN(MIN)/2.7) – 1 these set the absolute minimum working voltage, if the cells can't source the required power the switcher will supply the max current to keep Vin_reg > 2.7V currently set to 6V will need changed"
- note removed: "add more i/p's for cells in series/ parallel"
- note removed: "implement mppt with solar telem's"
Changed lines of the file:
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@@
     (effects (font (size 1.27 1.27)) (justify left bottom))
   )
-  (text "RIN1/RIN2 = (VIN(MIN)/2.7) – 1\nthese set the absolute minimum working voltage,\nif the cells can't source the required power the switcher will \nsupply the max current to keep Vin_reg > 2.7V\ncurrently set to 6V will need changed"
-    (at 86.36 57.15 0)
+  (text "RIN1/RIN2 = (VIN(MIN)/2.7) – 1\nthese set the MPP for the cells"
+    (at 86.36 49.53 0)
     (effects (font (size 1.27 1.27)) (justify left bottom))
   )
@@
     (effects (font (size 1.27 1.27)) (justify left bottom))
   )
-  (text "add more i/p's for cells in series/ parallel" (at 1.27 69.85 0)
-    (effects (font (size 1.27 1.27)) (justify left bottom))
-  )
-  (text "implement mppt with solar telem's" (at 19.05 96.52 0)
-    (effects (font (size 1.27 1.27) (thickness 0.254) bold) (justify left bottom))
-  )
   (text "rsense = 0.1/(ichgmax)" (at 184.15 60.96 0)

Commit message: em design complete
todo: update BOM
Parts:
- L203: footprint Inductor_SMD:L_Wuerth_WE-PD-Typ-LS -> mainboard-SLI:L_Wuerth_WE-PD-1260
- U211: footprint Package_SO:MSOP-12-1EP_3x4mm_P0.65mm_EP1.65x2.85mm_ThermalVias -> mainboard-SLI:MSOP-12-1EP_3x4mm_P0.65mm_EP1.65x2.85mm_ThermalVias
Changed lines of the file:
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@@
     (property "Reference" "U211" (id 0) (at 131.445 69.469 0))
     (property "Value" "‎LT3652HVEMSE#TRPBF‎" (id 1) (at 131.445 71.7804 0))
-    (property "Footprint" "Package_SO:MSOP-12-1EP_3x4mm_P0.65mm_EP1.65x2.85mm_ThermalVias" (id 2) (at 132.08 73.66 0)
+    (property "Footprint" "mainboard-SLI:MSOP-12-1EP_3x4mm_P0.65mm_EP1.65x2.85mm_ThermalVias" (id 2) (at 132.08 73.66 0)
       (effects (font (size 1.27 1.27)) hide)
     )
@@
     (property "Reference" "L203" (id 0) (at 182.88 63.754 90))
     (property "Value" "22uH" (id 1) (at 182.88 66.0654 90))
-    (property "Footprint" "Inductor_SMD:L_Wuerth_WE-PD-Typ-LS" (id 2) (at 182.88 68.58 0)
+    (property "Footprint" "mainboard-SLI:L_Wuerth_WE-PD-1260" (id 2) (at 182.88 68.58 0)
       (effects (font (size 1.27 1.27)) hide)
     )
