File: hardware/foras-promineo-revB-em/SLI-Backplane-Blank-Card-KiCad.kicad_sch (KiCad schematic)
At the start: 31 parts, among them P1 Card Edge for HSEC8-160-01-S-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, Q10 MMBT3906-7-F, Q207 IRF7404, Q208 IRF7458, Q211 IRF7404, Q212 IRF7404, Q213 IRF7404, Q220 IRF7404, Q51 MMBT4401-7-F, Q52 MMBT3906-7-F, Q53 MMBT3906-7-F, Q54 MMBT3906-7-F, Q9 MMBT3906-7-F

Commit message: swapped sda and scl output to bus :(
Connections:
- net SCL: now also P1.93 (Pin93); no longer P1.89 (Pin_89)
- net SDA: now also P1.89 (Pin_89); no longer P1.93 (Pin93)
Changed lines of the file:
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@@
-    )
-  )
-  (global_label "SDA" (shape bidirectional) (at 142.24 152.4 0) (fields_autoplaced)
-    (effects (font (size 1.27 1.27)) (justify left))
-    (property "Intersheet References" "${INTERSHEET_REFS}" (id 0) (at 0 0 0)
-      (effects (font (size 1.27 1.27)) hide)
     )
   )
@@
     )
   )
-  (global_label "SCL" (shape input) (at 142.24 148.59 0) (fields_autoplaced)
-    (effects (font (size 1.27 1.27)) (justify left))
-    (property "Intersheet References" "${INTERSHEET_REFS}" (id 0) (at 0 0 0)
-      (effects (font (size 1.27 1.27)) hide)
-    )
-  )
   (global_label "VBUS_INHIBIT" (shape bidirectional) (at 251.46 64.77 180) (fields_autoplaced)
     (effects (font (size 1.27 1.27)) (justify right))
@@
     (effects (font (size 1.27 1.27)) (justify right))
     (property "Intersheet References" "${INTERSHEET_REFS}" (id 0) (at 0 0 0)
+      (effects (font (size 1.27 1.27)) hide)
+    )
+  )
+  (global_label "SCL" (shape input) (at 142.24 152.4 0) (fields_autoplaced)
+    (effects (font (size 1.27 1.27)) (justify left))
+    (property "Intersheet References" "${INTERSHEET_REFS}" (id 0) (at 0 3.81 0)
       (effects (font (size 1.27 1.27)) hide)
     )
@@
       (effects (font (size 1.27 1.27)) hide)
     )
+  )
+  (global_label "SDA" (shape bidirectional) (at 142.24 148.59 0) (fields_autoplaced)
+    (effects (font (size 1.27 1.27)) (justify left))
+    (property "Intersheet References" "${INTERSHEET_REFS}" (id 0) (at 0 -3.81 0)
+      (effects (font (size 1.27 1.27)) hide)
+    )

Commit message: em design complete
todo: update BOM
Parts:
- added C52, C53: 0.1uF, Capacitor_SMD:C_0603_1608Metric, symbol Device:C
- added C54: 0.01uF, Capacitor_SMD:C_0603_1608Metric, symbol Device:C
- added R136, R137, R138, R139, R140, R141, R142, R143, R144, R145, R146, R147, R148, R149, R150, R151, R153, R154, R155, R156, R157, R158, R159, R160, R161, R162, R163, R164, R165: 330, Resistor_SMD:R_0603_1608Metric, symbol Device:R_US
- added R152, R166: 2.7k, Resistor_SMD:R_0603_1608Metric, symbol Device:R_US
- added U51: LTC4307, Package_SO:MSOP-8_3x3mm_P0.65mm, symbol mainboard_SLI:LTC4307
- added U52, U53: SN74LVCH245APWR, Package_SO:TSSOP-20_4.4x6.5mm_P0.65mm, symbol mainboard_SLI:SN74LVCH245APWR
Connections:
- net H1-4 is gone; now on net PC03: P1.14 (Pin_14)
- net 3.3V: now also C52.1, C53.1, C54.1, R136.1, R152.1, R166.1, U51.8 (VCC), U52.20 (V_{CC}), U53.20 (V_{CC})
- net AIN7: now also P1.24 (Pin_24)
- net GND: now also C52.2, C53.2, C54.2, R137.1, R147.1, R148.1, R149.1, R150.1, R151.1, R157.2, R158.2, R159.2, R160.2, U51.4 (GND), U52.10 (GND), U53.10 (GND)
- net MISO: now also R138.1; no longer P1.50 (Pin_50)
- net MOSI: now also R142.1; no longer P1.53 (Pin_53)
- net PC03: no longer P1.24 (Pin_24)
- net RX_MCU_2: now also R139.1; no longer P1.45 (Pin_45)
- net RX_MCU_3: now also R140.1; no longer P1.85 (Pin_85)
- net RX_MCU_4: now also R141.1; no longer P1.41 (Pin_41)
- net SCK: now also R143.1; no longer P1.49 (Pin_49)
- net SCL: now also U51.3 (SCLIN); no longer P1.93 (Pin93)
- net SDA: now also U51.6 (SDAIN); no longer P1.89 (Pin_89)
- net TX_MCU_2: now also R144.1; no longer P1.46 (Pin_46)
- net TX_MCU_3: now also R145.1; no longer P1.86 (Pin_86)
- net TX_MCU_4: now also R146.1; no longer P1.42 (Pin_42)
- new net: R162.1, U52.17 (B2)
- new net: R157.1, U53.14 (B5)
- new net: R154.1, U53.17 (B2)
- new net: R145.2, U52.5 (A4)
- new net: R148.2, U52.8 (A7)
- new net: R163.1, U52.16 (B3)
- new net: R146.2, U52.6 (A5)
- new net: R136.2, U52.1 (DIR)
- new net: R138.2, U53.2 (A1)
- new net: R137.2, U52.19 (~{OE})
- new net: R141.2, U53.5 (A4)
- new net: R165.1, U52.14 (B5)
- new net: R164.1, U52.15 (B4)
- new net: R149.2, U52.9 (A8)
- new net: R140.2, U53.4 (A3)
- new net: R144.2, U52.4 (A3)
- new net: R155.1, U53.16 (B3)
- new net: R161.1, U52.18 (B1)
- new net: R142.2, U52.2 (A1)
- new net: R143.2, U52.3 (A2)
- new net: R147.2, U52.7 (A6)
- new net: R156.1, U53.15 (B4)
- new net: R160.1, U53.11 (B8)
- new net: R159.1, U53.12 (B7)
- new net: R151.2, U53.19 (~{OE})
- new net: R150.2, U53.1 (DIR)
- new net: R158.1, U53.13 (B6)
- new net: R153.1, U53.18 (B1)
- new net: R139.2, U53.3 (A2)
- new net H1-17: P1.41 (Pin_41), R156.2
- new net H1-18: P1.42 (Pin_42), R165.2
- new net H1-19: P1.45 (Pin_45), R154.2
- new net H1-20: P1.46 (Pin_46), R163.2
- new net H1-21: P1.49 (Pin_49), R162.2
- new net H1-22: P1.50 (Pin_50), R153.2
- new net H1-23: P1.53 (Pin_53), R161.2
- new net H1-39: P1.85 (Pin_85), R155.2
- new net H1-40: P1.86 (Pin_86), R164.2
- new net H1-41: P1.89 (Pin_89), R166.2, U51.7 (SDAOUT)
- new net H1-43: P1.93 (Pin93), R152.2, U51.2 (SCLOUT)
- no-connect marks 1 -> 8
Other:
- note added: "40Vmax"
- note added: "5V @2A max"
- note added: "5V @3A max"
- note added: "GPIO can also be UART FC"
- note added: "backplane LED's"
- note added: "possibly move these to microJSTs?"
- note added: "unused"
- note removed: "5V @2A capacity with the switcher otherwise 1.5A (using linear regulator)"
- note removed: "<< not implemented"
- note removed: "Data"
- note removed: "Irridium UART"
- note removed: "NTC needs to be added to batt board"
- note removed: "Rx"
- note removed: "Tx"
- note removed: "if reconfigured as i2c, slave needs to have pull-ups"
- note removed: "openLST UART"
- note removed: "per my calculations, full power consumption exceeds USB's capabilities."
- note removed: "possible move these to microJSTs?"
- note removed: "spi bus -- not currently used by any other cards"
- note removed: "the pull ups on the backplane need to be DNP"
- note removed: "uart bus to the openMV H7 module"
- note removed: "unused currently open drain"
- note removed: "unused currently pulled low"

Commit message: real em commit
Connections:
- net 3.3V: now also U51.1 (EN)
Changed lines of the file:
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@@
   (junction (at 360.68 52.07) (diameter 0) (color 0 0 0 0)
+  )
+  (junction (at 152.4 163.83) (diameter 0) (color 0 0 0 0)
   )
   (junction (at 132.08 213.36) (diameter 0) (color 0 0 0 0)
@@
     (stroke (width 0) (type default) (color 0 0 0 0))
   )
+  (wire (pts (xy 152.4 163.83) (xy 152.4 167.64))
+    (stroke (width 0) (type default) (color 0 0 0 0))
+  )
